File: Design/BalancingBusinessCard/LIS3DHTR.sch (KiCad schematic (older format))
At the start: 3 parts

Commit message: Assigned numbers
Parts:
- gave numbers to parts that had none: 3
Changed lines of the file:
@@
 $EndDescr
 $Comp
-L Custom:LIS3DHTR U?
+L Custom:LIS3DHTR U401
 U 1 1 5BCBF7EE
 P 4250 2100
-F 0 "U?" H 5750 2593 60  0000 C CNN
+F 0 "U401" H 5750 2593 60  0000 C CNN
 F 1 "LIS3DHTR" H 5750 2487 60  0000 C CNN
 F 2 "LGA-16_3x3x1mm" H 5750 2340 60  0001 C CNN
@@
 $EndComp
 $Comp
-L power:+1V8 #PWR?
+L power:+1V8 #PWR0126
 U 1 1 5BCBF991
 P 4250 2100
-F 0 "#PWR?" H 4250 1950 50  0001 C CNN
+F 0 "#PWR0126" H 4250 1950 50  0001 C CNN
 F 1 "+1V8" H 4265 2273 50  0000 C CNN
 F 2 "" H 4250 2100 50  0001 C CNN
@@
 SCL
 $Comp
-L power:GND #PWR?
+L power:GND #PWR0127
 U 1 1 5BCBFB95
 P 4250 2500
-F 0 "#PWR?" H 4250 2250 50  0001 C CNN
+F 0 "#PWR0127" H 4250 2250 50  0001 C CNN
 F 1 "GND" V 4255 2372 50  0000 R CNN
 F 2 "" H 4250 2500 50  0001 C CNN
@@
 $EndComp
 $Comp
-L power:+1V8 #PWR?
+L power:+1V8 #PWR0128
 U 1 1 5BCBFC28
 P 4250 2800
-F 0 "#PWR?" H 4250 2650 50  0001 C CNN
+F 0 "#PWR0128" H 4250 2650 50  0001 C CNN
 F 1 "+1V8" V 4265 2928 50  0000 L CNN
 F 2 "" H 4250 2800 50  0001 C CNN
@@
 $EndComp
 $Comp
-L power:GND #PWR?
+L power:GND #PWR0129
 U 1 1 5BCBFCA0
 P 4250 2700
-F 0 "#PWR?" H 4250 2450 50  0001 C CNN
+F 0 "#PWR0129" H 4250 2450 50  0001 C CNN
 F 1 "GND" V 4255 2572 50  0000 R CNN
 F 2 "" H 4250 2700 50  0001 C CNN
@@
 $EndComp
 $Comp
-L power:GND #PWR?
+L power:GND #PWR0130
 U 1 1 5BCBFE0D
 P 7250 2500
-F 0 "#PWR?" H 7250 2250 50  0001 C CNN
+F 0 "#PWR0130" H 7250 2250 50  0001 C CNN
 F 1 "GND" V 7255 2372 50  0000 R CNN
 F 2 "" H 7250 2500 50  0001 C CNN
@@
 $EndComp
 $Comp
-L power:GND #PWR?
+L power:GND #PWR0131
 U 1 1 5BCBFE24
 P 7250 2700
-F 0 "#PWR?" H 7250 2450 50  0001 C CNN
+F 0 "#PWR0131" H 7250 2450 50  0001 C CNN
 F 1 "GND" V 7255 2572 50  0000 R CNN
 F 2 "" H 7250 2700 50  0001 C CNN
@@
 NoConn ~ 7250 2100
 $Comp
-L Device:C C?
+L Device:C C401
 U 1 1 5BCC04AB
 P 7800 2450
-F 0 "C?" H 7915 2496 50  0000 L CNN
+F 0 "C401" H 7915 2496 50  0000 L CNN
 F 1 "10uF" H 7915 2405 50  0000 L CNN
 F 2 "" H 7838 2300 50  0001 C CNN
@@
 $EndComp
 $Comp
-L Device:C C?
+L Device:C C402
 U 1 1 5BCC04F1
 P 8100 2450
-F 0 "C?" H 8215 2496 50  0000 L CNN
+F 0 "C402" H 8215 2496 50  0000 L CNN
 F 1 "100nF" H 8215 2405 50  0000 L CNN
 F 2 "" H 8138 2300 50  0001 C CNN
@@
 	7800 2600 7950 2600
 $Comp
-L power:GND #PWR?
+L power:GND #PWR0132
 U 1 1 5BCC05A4
 P 7950 2600
-F 0 "#PWR?" H 7950 2350 50  0001 C CNN
+F 0 "#PWR0132" H 7950 2350 50  0001 C CNN
 F 1 "GND" H 7955 2427 50  0000 C CNN
 F 2 "" H 7950 2600 50  0001 C CNN
@@
 	7950 2600 8100 2600
 $Comp
-L power:+1V8 #PWR?
+L power:+1V8 #PWR0133
 U 1 1 5BCC05FF
 P 8100 2300
-F 0 "#PWR?" H 8100 2150 50  0001 C CNN
+F 0 "#PWR0133" H 8100 2150 50  0001 C CNN
 F 1 "+1V8" H 8115 2473 50  0000 C CNN
 F 2 "" H 8100 2300 50  0001 C CNN
