File: Design/BalancingBusinessCard/ft550.sch (KiCad schematic (older format))
At the start: 7 parts, among them U501 FT440CA

Commit message: Made battery and circle centered and added edge cuts
Parts:
- C501, C502: footprint Capacitor_SMD:C_0603_1608Metric -> (none)
- C503: footprint Capacitor_SMD:C_0805_2012Metric -> (none)
- L501: footprint Inductor_SMD:L_0805_2012Metric -> (none)
- R501, R502: footprint Resistor_SMD:R_0603_1608Metric -> (none)
- U501: footprint Package_TO_SOT_SMD:SOT-23-5 -> FRE_SOT23-5
Changed lines of the file:
@@
 F 0 "C501" H 4415 3146 50  0000 L CNN
 F 1 "4.7uF" H 4415 3055 50  0000 L CNN
-F 2 "Capacitor_SMD:C_0603_1608Metric" H 4338 2950 50  0001 C CNN
+F 2 "" H 4338 2950 50  0001 C CNN
 F 3 "~" H 4300 3100 50  0001 C CNN
 	1    4300 3100
@@
 F 0 "U501" H 5700 3337 60  0000 C CNN
 F 1 "FT440CA" H 5700 3231 60  0000 C CNN
-F 2 "Package_TO_SOT_SMD:SOT-23-5" H 5700 3190 60  0001 C CNN
+F 2 "FRE_SOT23-5" H 5700 3190 60  0001 C CNN
 F 3 "" H 4600 2950 60  0000 C CNN
 	1    4600 2950
@@
 F 0 "L501" V 7340 3150 50  0000 C CNN
 F 1 "2.2uH" V 7249 3150 50  0000 C CNN
-F 2 "Inductor_SMD:L_0805_2012Metric" H 7150 3150 50  0001 C CNN
+F 2 "" H 7150 3150 50  0001 C CNN
 F 3 "~" H 7150 3150 50  0001 C CNN
 	1    7150 3150
@@
 F 0 "C503" H 7665 3446 50  0000 L CNN
 F 1 "10uF" H 7665 3355 50  0000 L CNN
-F 2 "Capacitor_SMD:C_0805_2012Metric" H 7588 3250 50  0001 C CNN
+F 2 "" H 7588 3250 50  0001 C CNN
 F 3 "~" H 7550 3400 50  0001 C CNN
 	1    7550 3400
@@
 F 0 "R501" H 6870 2646 50  0000 L CNN
 F 1 "100k" H 6870 2555 50  0000 L CNN
-F 2 "Resistor_SMD:R_0603_1608Metric" V 6730 2600 50  0001 C CNN
+F 2 "" V 6730 2600 50  0001 C CNN
 F 3 "~" H 6800 2600 50  0001 C CNN
 	1    6800 2600
@@
 F 0 "C502" V 6998 2600 50  0000 C CNN
 F 1 "22pF" V 7089 2600 50  0000 C CNN
-F 2 "Capacitor_SMD:C_0603_1608Metric" H 7288 2450 50  0001 C CNN
+F 2 "" H 7288 2450 50  0001 C CNN
 F 3 "~" H 7250 2600 50  0001 C CNN
 	1    7250 2600
@@
 F 0 "R502" V 7150 2750 50  0000 C CNN
 F 1 "200k" V 7250 2750 50  0000 C CNN
-F 2 "Resistor_SMD:R_0603_1608Metric" V 7180 2750 50  0001 C CNN
+F 2 "" V 7180 2750 50  0001 C CNN
 F 3 "~" H 7250 2750 50  0001 C CNN
 	1    7250 2750

Commit message: Final schematic assignments
Parts:
- C501, C502: footprint (none) -> Capacitor_SMD:C_0603_1608Metric
- C503: footprint (none) -> Capacitor_SMD:C_0805_2012Metric
- L501: footprint (none) -> Inductor_SMD:L_0805_2012Metric
- R501, R502: footprint (none) -> Resistor_SMD:R_0603_1608Metric
- U501: footprint FRE_SOT23-5 -> Package_TO_SOT_SMD:SOT-23-5
Changed lines of the file:
@@
 F 0 "C501" H 4415 3146 50  0000 L CNN
 F 1 "4.7uF" H 4415 3055 50  0000 L CNN
-F 2 "" H 4338 2950 50  0001 C CNN
+F 2 "Capacitor_SMD:C_0603_1608Metric" H 4338 2950 50  0001 C CNN
 F 3 "~" H 4300 3100 50  0001 C CNN
 	1    4300 3100
@@
 F 0 "U501" H 5700 3337 60  0000 C CNN
 F 1 "FT440CA" H 5700 3231 60  0000 C CNN
-F 2 "FRE_SOT23-5" H 5700 3190 60  0001 C CNN
+F 2 "Package_TO_SOT_SMD:SOT-23-5" H 5700 3190 60  0001 C CNN
 F 3 "" H 4600 2950 60  0000 C CNN
 	1    4600 2950
@@
 F 0 "L501" V 7340 3150 50  0000 C CNN
 F 1 "2.2uH" V 7249 3150 50  0000 C CNN
-F 2 "" H 7150 3150 50  0001 C CNN
+F 2 "Inductor_SMD:L_0805_2012Metric" H 7150 3150 50  0001 C CNN
 F 3 "~" H 7150 3150 50  0001 C CNN
 	1    7150 3150
@@
 F 0 "C503" H 7665 3446 50  0000 L CNN
 F 1 "10uF" H 7665 3355 50  0000 L CNN
-F 2 "" H 7588 3250 50  0001 C CNN
+F 2 "Capacitor_SMD:C_0805_2012Metric" H 7588 3250 50  0001 C CNN
 F 3 "~" H 7550 3400 50  0001 C CNN
 	1    7550 3400
@@
 F 0 "R501" H 6870 2646 50  0000 L CNN
 F 1 "100k" H 6870 2555 50  0000 L CNN
-F 2 "" V 6730 2600 50  0001 C CNN
+F 2 "Resistor_SMD:R_0603_1608Metric" V 6730 2600 50  0001 C CNN
 F 3 "~" H 6800 2600 50  0001 C CNN
 	1    6800 2600
@@
 F 0 "C502" V 6998 2600 50  0000 C CNN
 F 1 "22pF" V 7089 2600 50  0000 C CNN
-F 2 "" H 7288 2450 50  0001 C CNN
+F 2 "Capacitor_SMD:C_0603_1608Metric" H 7288 2450 50  0001 C CNN
 F 3 "~" H 7250 2600 50  0001 C CNN
 	1    7250 2600
@@
 F 0 "R502" V 7150 2750 50  0000 C CNN
 F 1 "200k" V 7250 2750 50  0000 C CNN
-F 2 "" V 7180 2750 50  0001 C CNN
+F 2 "Resistor_SMD:R_0603_1608Metric" V 7180 2750 50  0001 C CNN
 F 3 "~" H 7250 2750 50  0001 C CNN
 	1    7250 2750
