File: Design/BalancingBusinessCard/ft550.sch (KiCad schematic (older format))
At the start: 7 parts, among them U501 FT440CA

Commit message: Got Schematic CRC running
Changed lines of the file:
@@
 Wire Wire Line
 	7400 3150 7550 3150
+$Comp
+L power:PWR_FLAG #FLG0103
+U 1 1 5BCCA913
+P 7550 3150
+F 0 "#FLG0103" H 7550 3225 50  0001 C CNN
+F 1 "PWR_FLAG" H 7550 3324 50  0000 C CNN
+F 2 "" H 7550 3150 50  0001 C CNN
+F 3 "~" H 7550 3150 50  0001 C CNN
+	1    7550 3150
+	1    0    0    -1
+$EndComp
+Connection ~ 7550 3150
 $EndSCHEMATC

Commit message: Programming starting
Parts:
- removed C502: 22pF, symbol Device:C
- removed R501: 100k, symbol Device:R
- removed R502: 200k, symbol Device:R
Connections:
- wire segments 13 -> 10
Changed lines of the file:
@@
 	7000 3150 6800 3150
-Wire Wire Line
-	7300 3150 7400 3150
 Wire Wire Line
 	7550 3150 7550 3250
@@
 Wire Wire Line
 	6800 2950 6800 2750
-Wire Wire Line
-	6800 2750 7100 2750
-Wire Wire Line
-	7100 2750 7100 2600
-$Comp
-L Device:R R501
-U 1 1 5BCC4CF2
-P 6800 2600
-F 0 "R501" H 6870 2646 50  0000 L CNN
-F 1 "100k" H 6870 2555 50  0000 L CNN
-F 2 "" V 6730 2600 50  0001 C CNN
-F 3 "~" H 6800 2600 50  0001 C CNN
-	1    6800 2600
-	1    0    0    -1
-$EndComp
-Connection ~ 6800 2750
-Wire Wire Line
-	6800 2450 6650 2450
-$Comp
-L power:GND #PWR0502
-U 1 1 5BCC4E33
-P 6650 2450
-F 0 "#PWR0502" H 6650 2200 50  0001 C CNN
-F 1 "GND" H 6655 2277 50  0000 C CNN
-F 2 "" H 6650 2450 50  0001 C CNN
-F 3 "" H 6650 2450 50  0001 C CNN
-	1    6650 2450
-	1    0    0    -1
-$EndComp
-$Comp
-L Device:C C502
-U 1 1 5BCC4E79
-P 7250 2600
-F 0 "C502" V 6998 2600 50  0000 C CNN
-F 1 "22pF" V 7089 2600 50  0000 C CNN
-F 2 "" H 7288 2450 50  0001 C CNN
-F 3 "~" H 7250 2600 50  0001 C CNN
-	1    7250 2600
-	0    1    1    0
-$EndComp
-$Comp
-L Device:R R502
-U 1 1 5BCC4F31
-P 7250 2750
-F 0 "R502" V 7150 2750 50  0000 C CNN
-F 1 "200k" V 7250 2750 50  0000 C CNN
-F 2 "" V 7180 2750 50  0001 C CNN
-F 3 "~" H 7250 2750 50  0001 C CNN
-	1    7250 2750
-	0    -1   -1   0
-$EndComp
-Connection ~ 7100 2750
-Wire Wire Line
-	7400 2600 7400 2750
-Wire Wire Line
-	7400 2750 7400 3150
-Connection ~ 7400 2750
-Connection ~ 7400 3150
-Wire Wire Line
-	7400 3150 7550 3150
 $Comp
 L power:PWR_FLAG #FLG0103
@@
 $EndComp
 Connection ~ 7550 3150
+Wire Wire Line
+	7300 3150 7350 3150
+Wire Wire Line
+	7350 2750 7350 3150
+Wire Wire Line
+	6800 2750 7350 2750
+Connection ~ 7350 3150
+Wire Wire Line
+	7350 3150 7550 3150
 $EndSCHEMATC
