File: Design/BalancingBusinessCard/motorModule.sch (KiCad schematic (older format))
At the start: 4 parts, among them M201 Motor_DC, U201 AP1017AEN

Commit message: Made battery and circle centered and added edge cuts
Parts:
- M201: footprint Connector_PinHeader_2.54mm:PinHeader_1x02_P2.54mm_Vertical -> (none)
Changed lines of the file:
@@
 F 0 "M201" V 4055 4600 50  0000 C CNN
 F 1 "Motor_DC" V 4146 4600 50  0000 C CNN
-F 2 "Connector_PinHeader_2.54mm:PinHeader_1x02_P2.54mm_Vertical" H 4350 4560 50  0001 C CNN
+F 2 "" H 4350 4560 50  0001 C CNN
 F 3 "~" H 4350 4560 50  0001 C CNN
 	1    4350 4650

Commit message: Final schematic assignments
Parts:
- M201: footprint (none) -> Connector_PinHeader_2.54mm:PinHeader_1x02_P2.54mm_Vertical
Changed lines of the file:
@@
 F 0 "M201" V 4055 4600 50  0000 C CNN
 F 1 "Motor_DC" V 4146 4600 50  0000 C CNN
-F 2 "" H 4350 4560 50  0001 C CNN
+F 2 "Connector_PinHeader_2.54mm:PinHeader_1x02_P2.54mm_Vertical" H 4350 4560 50  0001 C CNN
 F 3 "~" H 4350 4560 50  0001 C CNN
 	1    4350 4650
