File: Design/BalancingBusinessCard/BalancingBusinessCard.sch (KiCad schematic (older format))
At the start: 8 parts, among them J101 TestPoints, U101 ATtiny261-20SU

Commit message: Final schematic assignments
Parts:
- BT101: footprint (none) -> CustomFootprints:CR2016VP
Changed lines of the file:
@@
 F 0 "BT101" H 4508 1346 50  0000 L CNN
 F 1 "Battery" H 4508 1255 50  0000 L CNN
-F 2 "" V 4400 1360 50  0001 C CNN
+F 2 "CustomFootprints:CR2016VP" V 4400 1360 50  0001 C CNN
 F 3 "~" V 4400 1360 50  0001 C CNN
 	1    4400 1300

Commit message: Made battery and circle centered and added edge cuts
Parts:
- BT101: footprint CustomFootprints:CR2016VP -> (none)
Changed lines of the file:
@@
 F 0 "BT101" H 4508 1346 50  0000 L CNN
 F 1 "Battery" H 4508 1255 50  0000 L CNN
-F 2 "CustomFootprints:CR2016VP" V 4400 1360 50  0001 C CNN
+F 2 "" V 4400 1360 50  0001 C CNN
 F 3 "~" V 4400 1360 50  0001 C CNN
 	1    4400 1300
