File: Design/BalancingBusinessCard/BalancingBusinessCard.sch (KiCad schematic (older format))
At the start: 8 parts

Commit message: Fixed stuff
Connections:
- wire segments 20 -> 17
Changed lines of the file:
@@
 	1    0    0    -1
 $EndComp
-Text Label 4000 3850 0    50   ~ 0
+Text Label 4100 3850 0    50   ~ 0
 MOSI
-Wire Wire Line
-	4000 3850 3800 3850
-Text Label 4000 3950 0    50   ~ 0
+Text Label 4100 3950 0    50   ~ 0
 MISO
-Text Label 4000 4050 0    50   ~ 0
+Text Label 4100 4050 0    50   ~ 0
 SCK
-Wire Wire Line
-	4000 4050 3800 4050
-Wire Wire Line
-	4000 3950 3800 3950
 Text Label 7500 4200 2    50   ~ 0
 VCL
@@
 LED_8
 Wire Wire Line
-	3800 3850 4100 3850
-Wire Wire Line
-	4100 3950 3800 3950
-Wire Wire Line
-	3800 4050 4100 4050
-Wire Wire Line
 	3200 4850 3100 4850
 Connection ~ 3100 4850
@@
 	1    0    0    -1
 $EndComp
+Wire Wire Line
+	3800 3850 4100 3850
+Wire Wire Line
+	3800 4050 4100 4050
+Wire Wire Line
+	3800 3950 4100 3950
 $EndSCHEMATC

Commit message: Assigned numbers
Parts:
- gave numbers to parts that had none: 7
Connections:
- net LED_0: now also J101.5 (Pin_5)
- net LED_1: now also J101.6 (Pin_6)
- net LED_2: now also J101.7 (Pin_7)
- net LED_3: now also J101.8 (Pin_8)
Changed lines of the file:
@@
 $EndDescr
 $Comp
-L MCU_Microchip_ATtiny:ATtiny261A-SU U?
+L MCU_Microchip_ATtiny:ATtiny261A-SU U101
 U 1 1 5BCB9B43
 P 3100 3750
-F 0 "U?" H 2470 3796 50  0000 R CNN
+F 0 "U101" H 2470 3796 50  0000 R CNN
 F 1 "ATtiny261-20SU" H 2470 3705 50  0000 R CNN
 F 2 "Package_SO:SOIC-20W_7.5x12.8mm_P1.27mm" H 3100 3750 50  0001 C CIN
@@
 SCL
 $Comp
-L Device:Battery BT?
+L Device:Battery BT101
 U 1 1 5BCBEFF8
 P 4400 1300
-F 0 "BT?" H 4508 1346 50  0000 L CNN
+F 0 "BT101" H 4508 1346 50  0000 L CNN
 F 1 "Battery" H 4508 1255 50  0000 L CNN
 F 2 "" V 4400 1360 50  0001 C CNN
@@
 $EndComp
 $Comp
-L power:+BATT #PWR?
+L power:+BATT #PWR0101
 U 1 1 5BCBF44A
 P 4400 1050
-F 0 "#PWR?" H 4400 900 50  0001 C CNN
+F 0 "#PWR0101" H 4400 900 50  0001 C CNN
 F 1 "+BATT" H 4415 1223 50  0000 C CNN
 F 2 "" H 4400 1050 50  0001 C CNN
@@
 +3V
 $Comp
-L power:GND #PWR?
+L power:GND #PWR0102
 U 1 1 5BCBF4A9
 P 4400 1500
-F 0 "#PWR?" H 4400 1250 50  0001 C CNN
+F 0 "#PWR0102" H 4400 1250 50  0001 C CNN
 F 1 "GND" H 4405 1327 50  0000 C CNN
 F 2 "" H 4400 1500 50  0001 C CNN
@@
 $EndComp
 $Comp
-L power:+BATT #PWR?
+L power:+BATT #PWR0103
 U 1 1 5BCBF62A
 P 7050 4300
-F 0 "#PWR?" H 7050 4150 50  0001 C CNN
+F 0 "#PWR0103" H 7050 4150 50  0001 C CNN
 F 1 "+BATT" H 7065 4473 50  0000 C CNN
 F 2 "" H 7050 4300 50  0001 C CNN
@@
 MOSI
 $Comp
-L power:+1V8 #PWR?
+L power:+1V8 #PWR0104
 U 1 1 5BCBF021
 P 3300 5750
-F 0 "#PWR?" H 3300 5600 50  0001 C CNN
+F 0 "#PWR0104" H 3300 5600 50  0001 C CNN
 F 1 "+1V8" H 3315 5923 50  0000 C CNN
 F 2 "" H 3300 5750 50  0001 C CNN
@@
 $EndComp
 $Comp
-L Connector:Conn_01x10_Male J?
+L Connector:Conn_01x10_Male J101
 U 1 1 5BCBF241
 P 5150 6250
-F 0 "J?" V 5078 6177 50  0000 C CNN
+F 0 "J101" V 5078 6177 50  0000 C CNN
 F 1 "TestPoints" V 4987 6177 50  0000 C CNN
 F 2 "CustomFootprints:Testpoint_1x10" H 5150 6250 50  0001 C CNN
@@
 $EndComp
 $Comp
-L power:+1V8 #PWR?
+L power:+1V8 #PWR0105
 U 1 1 5BCBF527
 P 4850 6050
-F 0 "#PWR?" H 4850 5900 50  0001 C CNN
+F 0 "#PWR0105" H 4850 5900 50  0001 C CNN
 F 1 "+1V8" H 4865 6223 50  0000 C CNN
 F 2 "" H 4850 6050 50  0001 C CNN
@@
 $EndComp
 $Comp
-L power:+BATT #PWR?
+L power:+BATT #PWR0106
 U 1 1 5BCBF6B8
 P 4750 6050
-F 0 "#PWR?" H 4750 5900 50  0001 C CNN
+F 0 "#PWR0106" H 4750 5900 50  0001 C CNN
 F 1 "+BATT" H 4765 6223 50  0000 C CNN
 F 2 "" H 4750 6050 50  0001 C CNN
@@
 $EndComp
 $Comp
-L power:GND #PWR?
+L power:GND #PWR0107
 U 1 1 5BCBF839
 P 3300 5950
-F 0 "#PWR?" H 3300 5700 50  0001 C CNN
+F 0 "#PWR0107" H 3300 5700 50  0001 C CNN
 F 1 "GND" V 3305 5822 50  0000 R CNN
 F 2 "" H 3300 5950 50  0001 C CNN
@@
 RESET
 $Comp
-L power:GND #PWR?
+L power:GND #PWR0108
 U 1 1 5BCCA97D
 P 3100 4850
-F 0 "#PWR?" H 3100 4600 50  0001 C CNN
+F 0 "#PWR0108" H 3100 4600 50  0001 C CNN
 F 1 "GND" H 3105 4677 50  0000 C CNN
 F 2 "" H 3100 4850 50  0001 C CNN
@@
 	4400 1100 5150 1100
 $Comp
-L power:GND #PWR?
+L power:GND #PWR0109
 U 1 1 5BCC0AD3
 P 5150 1400
-F 0 "#PWR?" H 5150 1150 50  0001 C CNN
+F 0 "#PWR0109" H 5150 1150 50  0001 C CNN
 F 1 "GND" H 5155 1227 50  0000 C CNN
 F 2 "" H 5150 1400 50  0001 C CNN
@@
 	7500 1300 7350 1300
 $Comp
-L Device:R R?
+L Device:R R102
 U 1 1 5BCC12E2
 P 7350 1150
-F 0 "R?" H 7420 1196 50  0000 L CNN
+F 0 "R102" H 7420 1196 50  0000 L CNN
 F 1 "1k" H 7420 1105 50  0000 L CNN
 F 2 "" V 7280 1150 50  0001 C CNN
@@
 Connection ~ 7350 1300
 $Comp
-L power:+1V8 #PWR?
+L power:+1V8 #PWR0110
 U 1 1 5BCC13E8
 P 7200 1000
-F 0 "#PWR?" H 7200 850 50  0001 C CNN
+F 0 "#PWR0110" H 7200 850 50  0001 C CNN
 F 1 "+1V8" H 7215 1173 50  0000 C CNN
 F 2 "" H 7200 1000 50  0001 C CNN
@@
 Connection ~ 7200 1000
 $Comp
-L Device:R R?
+L Device:R R101
 U 1 1 5BCC14CF
 P 7100 1250
-F 0 "R?" H 6950 1350 50  0000 L CNN
+F 0 "R101" H 6950 1350 50  0000 L CNN
 F 1 "1k" H 6950 1250 50  0000 L CNN
 F 2 "" V 7030 1250 50  0001 C CNN
@@
 Connection ~ 4400 1100
 $Comp
-L Device:C C?
+L Device:C C102
 U 1 1 5BCC09EB
 P 5150 1250
-F 0 "C?" H 5265 1296 50  0000 L CNN
+F 0 "C102" H 5265 1296 50  0000 L CNN
 F 1 "10uF" H 5265 1205 50  0000 L CNN
 F 2 "" H 5188 1100 50  0001 C CNN
@@
 	3200 2650 3100 2650
 $Comp
-L power:+1V8 #PWR?
+L power:+1V8 #PWR0111
 U 1 1 5BCC0FB3
 P 3100 2400
-F 0 "#PWR?" H 3100 2250 50  0001 C CNN
+F 0 "#PWR0111" H 3100 2250 50  0001 C CNN
 F 1 "+1V8" H 3115 2573 50  0000 C CNN
 F 2 "" H 3100 2400 50  0001 C CNN
@@
 Connection ~ 3100 2400
 $Comp
-L Device:C C?
+L Device:C C101
 U 1 1 5BCC392A
 P 3600 2400
-F 0 "C?" V 3852 2400 50  0000 C CNN
+F 0 "C101" V 3852 2400 50  0000 C CNN
 F 1 "10uF" V 3761 2400 50  0000 C CNN
 F 2 "" H 3638 2250 50  0001 C CNN
@@
 $EndComp
 $Comp
-L power:GND #PWR?
+L power:GND #PWR0112
 U 1 1 5BCC3A23
 P 3750 2400
-F 0 "#PWR?" H 3750 2150 50  0001 C CNN
+F 0 "#PWR0112" H 3750 2150 50  0001 C CNN
 F 1 "GND" H 3755 2227 50  0000 C CNN
 F 2 "" H 3750 2400 50  0001 C CNN
@@
 Wire Wire Line
 	3800 3950 4100 3950
+Text Label 5150 6050 1    50   ~ 0
+LED_0
+Text Label 5250 6050 1    50   ~ 0
+LED_1
+Text Label 5350 6050 1    50   ~ 0
+LED_2
+Text Label 5450 6050 1    50   ~ 0
+LED_3
 $EndSCHEMATC

Commit message: Footprint assignment
Parts:
- C101, C102: footprint (none) -> Capacitor_SMD:C_0805_2012Metric
- R101, R102: footprint (none) -> Resistor_SMD:R_0603_1608Metric
Changed lines of the file:
@@
 F 0 "R102" H 7420 1196 50  0000 L CNN
 F 1 "1k" H 7420 1105 50  0000 L CNN
-F 2 "" V 7280 1150 50  0001 C CNN
+F 2 "Resistor_SMD:R_0603_1608Metric" V 7280 1150 50  0001 C CNN
 F 3 "~" H 7350 1150 50  0001 C CNN
 	1    7350 1150
@@
 F 0 "R101" H 6950 1350 50  0000 L CNN
 F 1 "1k" H 6950 1250 50  0000 L CNN
-F 2 "" V 7030 1250 50  0001 C CNN
+F 2 "Resistor_SMD:R_0603_1608Metric" V 7030 1250 50  0001 C CNN
 F 3 "~" H 7100 1250 50  0001 C CNN
 	1    7100 1250
@@
 F 0 "C102" H 5265 1296 50  0000 L CNN
 F 1 "10uF" H 5265 1205 50  0000 L CNN
-F 2 "" H 5188 1100 50  0001 C CNN
+F 2 "Capacitor_SMD:C_0805_2012Metric" H 5188 1100 50  0001 C CNN
 F 3 "~" H 5150 1250 50  0001 C CNN
 	1    5150 1250
@@
 F 0 "C101" V 3852 2400 50  0000 C CNN
 F 1 "10uF" V 3761 2400 50  0000 C CNN
-F 2 "" H 3638 2250 50  0001 C CNN
+F 2 "Capacitor_SMD:C_0805_2012Metric" H 3638 2250 50  0001 C CNN
 F 3 "~" H 3600 2400 50  0001 C CNN
 	1    3600 2400

Commit message: Added regulator
Connections:
- wire segments 17 -> 21
Changed lines of the file:
@@
 $Descr A4 11693 8268
 encoding utf-8
-Sheet 1 4
+Sheet 1 5
 Title ""
 Date ""
@@
 Text Label 5450 6050 1    50   ~ 0
 LED_3
+$Comp
+L power:PWR_FLAG #FLG0101
+U 1 1 5BCC0D87
+P 4050 1100
+F 0 "#FLG0101" H 4050 1175 50  0001 C CNN
+F 1 "PWR_FLAG" H 4050 1274 50  0000 C CNN
+F 2 "" H 4050 1100 50  0001 C CNN
+F 3 "~" H 4050 1100 50  0001 C CNN
+	1    4050 1100
+	1    0    0    -1
+$EndComp
+Wire Wire Line
+	4050 1100 4400 1100
+$Comp
+L power:PWR_FLAG #FLG0102
+U 1 1 5BCC114E
+P 4050 1400
+F 0 "#FLG0102" H 4050 1475 50  0001 C CNN
+F 1 "PWR_FLAG" H 4050 1574 50  0000 C CNN
+F 2 "" H 4050 1400 50  0001 C CNN
+F 3 "~" H 4050 1400 50  0001 C CNN
+	1    4050 1400
+	1    0    0    -1
+$EndComp
+Wire Wire Line
+	4050 1450 4050 1400
+$Comp
+L power:GND #PWR0134
+U 1 1 5BCC13FA
+P 4050 1450
+F 0 "#PWR0134" H 4050 1200 50  0001 C CNN
+F 1 "GND" H 4055 1277 50  0000 C CNN
+F 2 "" H 4050 1450 50  0001 C CNN
+F 3 "" H 4050 1450 50  0001 C CNN
+	1    4050 1450
+	1    0    0    -1
+$EndComp
+$Sheet
+S 1050 800  1350 350
+U 5BCC40AE
+F0 "1v8 Regulator" 50
+F1 "ft550.sch" 50
+F2 "Vin" I R 2400 900 50
+F3 "Vout" I R 2400 1000 50
+$EndSheet
+$Comp
+L power:+BATT #PWR?
+U 1 1 5BCC563A
+P 2500 900
+F 0 "#PWR?" H 2500 750 50  0001 C CNN
+F 1 "+BATT" H 2515 1073 50  0000 C CNN
+F 2 "" H 2500 900 50  0001 C CNN
+F 3 "" H 2500 900 50  0001 C CNN
+	1    2500 900
+	1    0    0    -1
+$EndComp
+Wire Wire Line
+	2500 900  2400 900
+$Comp
+L power:+1V8 #PWR?
+U 1 1 5BCC5911
+P 2650 1000
+F 0 "#PWR?" H 2650 850 50  0001 C CNN
+F 1 "+1V8" H 2665 1173 50  0000 C CNN
+F 2 "" H 2650 1000 50  0001 C CNN
+F 3 "" H 2650 1000 50  0001 C CNN
+	1    2650 1000
+	1    0    0    -1
+$EndComp
+Wire Wire Line
+	2650 1000 2400 1000
 $EndSCHEMATC

Commit message: Programming starting
Parts:
- removed R101, R102: 1k, Resistor_SMD:R_0603_1608Metric, symbol Device:R
Connections:
- wire segments 21 -> 16
Changed lines of the file:
@@
 Text Label 7050 1400 2    50   ~ 0
 SCL
-Wire Wire Line
-	7500 1300 7350 1300
-$Comp
-L Device:R R102
-U 1 1 5BCC12E2
-P 7350 1150
-F 0 "R102" H 7420 1196 50  0000 L CNN
-F 1 "1k" H 7420 1105 50  0000 L CNN
-F 2 "Resistor_SMD:R_0603_1608Metric" V 7280 1150 50  0001 C CNN
-F 3 "~" H 7350 1150 50  0001 C CNN
-	1    7350 1150
-	1    0    0    -1
-$EndComp
-Wire Wire Line
-	7300 1300 7350 1300
-Connection ~ 7350 1300
-$Comp
-L power:+1V8 #PWR0110
-U 1 1 5BCC13E8
-P 7200 1000
-F 0 "#PWR0110" H 7200 850 50  0001 C CNN
-F 1 "+1V8" H 7215 1173 50  0000 C CNN
-F 2 "" H 7200 1000 50  0001 C CNN
-F 3 "" H 7200 1000 50  0001 C CNN
-	1    7200 1000
-	1    0    0    -1
-$EndComp
-Wire Wire Line
-	7350 1000 7200 1000
-Wire Wire Line
-	7200 1000 7100 1000
-Connection ~ 7200 1000
-$Comp
-L Device:R R101
-U 1 1 5BCC14CF
-P 7100 1250
-F 0 "R101" H 6950 1350 50  0000 L CNN
-F 1 "1k" H 6950 1250 50  0000 L CNN
-F 2 "Resistor_SMD:R_0603_1608Metric" V 7030 1250 50  0001 C CNN
-F 3 "~" H 7100 1250 50  0001 C CNN
-	1    7100 1250
-	1    0    0    -1
-$EndComp
-Wire Wire Line
-	7100 1000 7100 1100
-Wire Wire Line
-	7050 1400 7100 1400
-Wire Wire Line
-	7100 1400 7500 1400
-Connection ~ 7100 1400
 Text Label 7500 3800 2    50   ~ 0
 ADC0
@@
 Wire Wire Line
 	2650 1000 2400 1000
+Wire Wire Line
+	7300 1300 7500 1300
+Wire Wire Line
+	7050 1400 7500 1400
 $EndSCHEMATC
