File: Design/BalancingBusinessCard/BalancingBusinessCard.kicad_pcb (KiCad board)
At the start: 2 copper layers, 51 x 89 mm, 31 parts, among them J101 TestPoints, M201 Motor_DC, U101 ATtiny261-20SU, U201 AP1017AEN, U401 LIS3DHTR, U501 FT440CA

Commit message: Moved stuff
Parts:
- moved C202 21.1 mm to (191.1, 100.7), turned to 180 degrees
- moved C201 18.7 mm to (191.2, 104.7), turned to 180 degrees
Changed lines of the file:
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@@
   )
   (module Capacitor_SMD:C_0805_2012Metric (layer F.Cu)
-    (at 172.525001 105.605001)
+    (at 191.1625 104.7 180)
     (descr "Capacitor SMD 0805 (2012 Metric), square (rectangular) end terminal, IPC_7351 nominal, (Body size source: https://docs.google.com/spreadsheets/d/1BsfQQcO9C6DZCsRaXUlFlo91Tg2WpOkGARC1WS5S8t0/edit?usp=sharing), generated with kicad-footprint-generator")
     (tags capacitor)
     (attr smd)
-    (fp_text reference C201 (at 0 -1.65) (layer F.SilkS)
+    (fp_text reference C201 (at 0 -1.65 180) (layer F.SilkS)
       (effects (font (size 1 1) (thickness 0.15)))
     )
-    (fp_text value 10uF (at 0 1.65) (layer F.Fab)
+    (fp_text value 10uF (at 0 1.65 180) (layer F.Fab)
       (effects (font (size 1 1) (thickness 0.15)))
     )
-    (fp_text user %R (at 0 0) (layer F.Fab)
+    (fp_text user %R (at 0 0 180) (layer F.Fab)
       (effects (font (size 0.5 0.5) (thickness 0.08)))
     )
@@
     (fp_line (start -1 -0.6) (end 1 -0.6) (layer F.Fab) (width 0.1))
     (fp_line (start -1 0.6) (end -1 -0.6) (layer F.Fab) (width 0.1))
-    (pad 2 smd roundrect (at 0.9375 0) (size 0.975 1.4) (layers F.Cu F.Paste F.Mask) (roundrect_rratio 0.25)
+    (pad 2 smd roundrect (at 0.9375 0 180) (size 0.975 1.4) (layers F.Cu F.Paste F.Mask) (roundrect_rratio 0.25)
       (net 2 GND))
-    (pad 1 smd roundrect (at -0.9375 0) (size 0.975 1.4) (layers F.Cu F.Paste F.Mask) (roundrect_rratio 0.25)
+    (pad 1 smd roundrect (at -0.9375 0 180) (size 0.975 1.4) (layers F.Cu F.Paste F.Mask) (roundrect_rratio 0.25)
       (net 1 +BATT))
     (model ${KISYS3DMOD}/Capacitor_SMD.3dshapes/C_0805_2012Metric.wrl
@@
   )
   (module Capacitor_SMD:C_0603_1608Metric (layer F.Cu)
-    (at 172.0875 109.8)
+    (at 191.0875 100.7 180)
     (descr "Capacitor SMD 0603 (1608 Metric), square (rectangular) end terminal, IPC_7351 nominal, (Body size source: http://www.tortai-tech.com/upload/download/2011102023233369053.pdf), generated with kicad-footprint-generator")
     (tags capacitor)
     (attr smd)
-    (fp_text reference C202 (at 0 -1.43) (layer F.SilkS)
+    (fp_text reference C202 (at 0 -1.43 180) (layer F.SilkS)
       (effects (font (size 1 1) (thickness 0.15)))
     )
-    (fp_text value 1uF (at 0 1.43) (layer F.Fab)
+    (fp_text value 1uF (at 0 1.43 180) (layer F.Fab)
       (effects (font (size 1 1) (thickness 0.15)))
     )
-    (fp_text user %R (at 0 0) (layer F.Fab)
+    (fp_text user %R (at 0 0 180) (layer F.Fab)
       (effects (font (size 0.4 0.4) (thickness 0.06)))
     )
@@
     (fp_line (start -0.8 -0.4) (end 0.8 -0.4) (layer F.Fab) (width 0.1))
     (fp_line (start -0.8 0.4) (end -0.8 -0.4) (layer F.Fab) (width 0.1))
-    (pad 2 smd roundrect (at 0.7875 0) (size 0.875 0.95) (layers F.Cu F.Paste F.Mask) (roundrect_rratio 0.25)
+    (pad 2 smd roundrect (at 0.7875 0 180) (size 0.875 0.95) (layers F.Cu F.Paste F.Mask) (roundrect_rratio 0.25)
       (net 2 GND))
-    (pad 1 smd roundrect (at -0.7875 0) (size 0.875 0.95) (layers F.Cu F.Paste F.Mask) (roundrect_rratio 0.25)
+    (pad 1 smd roundrect (at -0.7875 0 180) (size 0.875 0.95) (layers F.Cu F.Paste F.Mask) (roundrect_rratio 0.25)
       (net 1 +BATT))
     (model ${KISYS3DMOD}/Capacitor_SMD.3dshapes/C_0603_1608Metric.wrl

Commit message: messiest of merges
Routing:
- net /LED_4: track 0.00 -> 59.3 mm
- net /LED_0: track 0.00 -> 55.8 mm, vias 0 -> 2
- net /LED_1: track 0.00 -> 50.8 mm, vias 0 -> 2
- net /LED_2: track 0.00 -> 47.6 mm
- net /LED_3: track 0.00 -> 44.5 mm
- net /MOSI: track 0.00 -> 34.1 mm, vias 0 -> 1
- net /SCK: track 0.00 -> 28.9 mm, vias 0 -> 2
- net /LED_5: track 0.00 -> 27.9 mm
- net /LED_6: track 0.00 -> 26.7 mm
- net +1V8: track 0.00 -> 25.3 mm, vias 0 -> 2
- net /LED_7: track 0.00 -> 23.0 mm
- net /LED_8: track 0.00 -> 19.2 mm
- net /RESET: track 0.00 -> 16.1 mm, vias 0 -> 1
- net /INB: track 0.00 -> 12.4 mm, vias 0 -> 2
- net /INA: track 0.00 -> 9.55 mm, vias 0 -> 2
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