File: Design/BalancingBusinessCard/BalancingBusinessCardMotor.sch (KiCad schematic (older format))
At the start: 6 parts, among them J101 TestPoints, U101 ATtiny261-20SU

Commit message: Completed Lights board schematic
Parts:
- C102: value 10uF -> 10uF 1%
Changed lines of the file:
@@
 EESchema Schematic File Version 4
-LIBS:BalancingBusinessCard-cache
 EELAYER 26 0
 EELAYER END
@@
 P 5150 1250
 F 0 "C102" H 5265 1296 50  0000 L CNN
-F 1 "10uF" H 5265 1205 50  0000 L CNN
+F 1 "10uF 1%" H 5265 1205 50  0000 L CNN
 F 2 "Capacitor_SMD:C_0805_2012Metric" H 5188 1100 50  0001 C CNN
 F 3 "~" H 5150 1250 50  0001 C CNN
