File: Design/BalancingBusinessCard/BalancingBusinessCardLights.sch (KiCad schematic (older format))
At the start: 14 parts, among them SW101 SW_SPST, U101 ATtiny261A-MU

Commit message: Finished light board layout and silkscreen design
Parts:
- removed C102: 10uF, Capacitor_SMD:C_0805_2012Metric, symbol Device:C
- removed TP101: BATT_TP, Measurement_Points:Measurement_Point_Round-SMD-Pad_Big, symbol Connector:Test_Point
- removed TP102: 3V3_TP, Measurement_Points:Measurement_Point_Round-SMD-Pad_Big, symbol Connector:Test_Point
- removed TP103: RESET_TP, Measurement_Points:Measurement_Point_Round-SMD-Pad_Big, symbol Connector:Test_Point
- removed TP104: LED_0_TP, Measurement_Points:Measurement_Point_Round-SMD-Pad_Big, symbol Connector:Test_Point
- removed TP105: LED_1_TP, Measurement_Points:Measurement_Point_Round-SMD-Pad_Big, symbol Connector:Test_Point
- removed TP106: LED_2_TP, Measurement_Points:Measurement_Point_Round-SMD-Pad_Big, symbol Connector:Test_Point
- removed TP107: TILT_TP, Measurement_Points:Measurement_Point_Round-SMD-Pad_Big, symbol Connector:Test_Point
- added R102, R103: 10k, Resistors_SMD:R_0603, symbol Device:R
- U101: footprint Package_DFN_QFN:QFN-32-1EP_5x5mm_P0.5mm_EP3.8x3.8mm -> Housings_DFN_QFN:QFN-32-1EP_5x5mm_Pitch0.5mm
Connections:
- net labels removed: VCL
- wire segments 35 -> 31
Changed lines of the file:
@@
 MOSI
-$Comp
-L power:+BATT #PWR0106
-U 1 1 5BCBF6B8
-P 4750 6050
-F 0 "#PWR0106" H 4750 5900 50  0001 C CNN
-F 1 "+BATT" V 4750 6300 50  0000 C CNN
-F 2 "" H 4750 6050 50  0001 C CNN
-F 3 "" H 4750 6050 50  0001 C CNN
-	1    4750 6050
-	1    0    0    -1
-$EndComp
 $Comp
 L power:GND #PWR0107
@@
 Text Label 3800 4550 0    50   ~ 0
 RESET
-Text Label 4950 6050 1    50   ~ 0
-RESET
 $Comp
 L power:GND #PWR0108
@@
 Text Label 4100 4050 0    50   ~ 0
 SCK
-Text Label 5150 1100 0    50   ~ 0
-VCL
-Wire Wire Line
-	4400 1100 5150 1100
-$Comp
-L power:GND #PWR0109
-U 1 1 5BCC0AD3
-P 5150 1400
-F 0 "#PWR0109" H 5150 1150 50  0001 C CNN
-F 1 "GND" H 5155 1227 50  0000 C CNN
-F 2 "" H 5150 1400 50  0001 C CNN
-F 3 "" H 5150 1400 50  0001 C CNN
-	1    5150 1400
-	1    0    0    -1
-$EndComp
 $Sheet
 S 7500 950  1600 1100
@@
 F3 "SCL" I L 7500 1400 50
 $EndSheet
-Text Label 7300 1300 2    50   ~ 0
+Text Label 7175 1300 2    50   ~ 0
 SDA
-Text Label 7050 1400 2    50   ~ 0
+Text Label 6825 1400 2    50   ~ 0
 SCL
 Wire Wire Line
 	4400 1100 4400 1050
 Connection ~ 4400 1100
-$Comp
-L Device:C C102
-U 1 1 5BCC09EB
-P 5150 1250
-F 0 "C102" H 5265 1296 50  0000 L CNN
-F 1 "10uF" H 5265 1205 50  0000 L CNN
-F 2 "Capacitor_SMD:C_0805_2012Metric" H 5188 1100 50  0001 C CNN
-F 3 "~" H 5150 1250 50  0001 C CNN
-	1    5150 1250
-	1    0    0    -1
-$EndComp
 Text Label 7500 2500 2    50   ~ 0
 LED_0
@@
 Text Label 3800 3650 0    50   ~ 0
 LED_4
+Text Label 3800 4450 0    50   ~ 0
+LED_5
+Text Label 3800 4350 0    50   ~ 0
+LED_6
+Text Label 3800 4250 0    50   ~ 0
+LED_7
 Text Label 3800 4150 0    50   ~ 0
-LED_5
-Text Label 3800 4250 0    50   ~ 0
-LED_6
-Text Label 3800 4350 0    50   ~ 0
-LED_7
-Text Label 3800 4450 0    50   ~ 0
 LED_8
 Wire Wire Line
@@
 Wire Wire Line
 	3800 3950 4100 3950
-Text Label 5050 6050 1    50   ~ 0
-LED_0
-Text Label 5150 6050 1    50   ~ 0
-LED_1
-Text Label 5250 6050 1    50   ~ 0
-LED_2
 $Comp
 L power:PWR_FLAG #FLG0101
@@
 	1    0    0    -1
 $EndComp
-Wire Wire Line
-	7300 1300 7500 1300
-Wire Wire Line
-	7050 1400 7500 1400
 $Comp
 L MCU_Microchip_ATtiny:ATtiny261A-MU U101
@@
 F 0 "U101" H 2459 3796 50  0000 R CNN
 F 1 "ATtiny261A-MU" H 2459 3705 50  0000 R CNN
-F 2 "Package_DFN_QFN:QFN-32-1EP_5x5mm_P0.5mm_EP3.8x3.8mm" H 3100 3750 50  0001 C CIN
+F 2 "Housings_DFN_QFN:QFN-32-1EP_5x5mm_Pitch0.5mm" H 3100 3750 50  0001 C CIN
 F 3 "http://ww1.microchip.com/downloads/en/DeviceDoc/doc8197.pdf" H 3100 3750 50  0001 C CNN
 	1    3100 3750
@@
 	1    0    0    -1
 $EndComp
-$Comp
-L power:+3V3 #PWR0111
-U 1 1 5C0EFBA3
-P 4850 6050
-F 0 "#PWR0111" H 4850 5900 50  0001 C CNN
-F 1 "+3V3" V 4850 6300 50  0000 C CNN
-F 2 "" H 4850 6050 50  0001 C CNN
-F 3 "" H 4850 6050 50  0001 C CNN
-	1    4850 6050
-	1    0    0    -1
-$EndComp
-$Comp
-L Connector:Test_Point TP101
-U 1 1 5C0F11B2
-P 4750 6225
-F 0 "TP101" V 4750 7025 50  0000 R CNN
-F 1 "BATT_TP" V 4750 6800 50  0000 R CNN
-F 2 "Measurement_Points:Measurement_Point_Round-SMD-Pad_Big" H 4950 6225 50  0001 C CNN
-F 3 "~" H 4950 6225 50  0001 C CNN
-	1    4750 6225
-	-1   0    0    1
-$EndComp
-Wire Wire Line
-	4750 6225 4750 6050
-$Comp
-L Connector:Test_Point TP102
-U 1 1 5C0F1679
-P 4850 6225
-F 0 "TP102" V 4850 7025 50  0000 R CNN
-F 1 "3V3_TP" V 4850 6800 50  0000 R CNN
-F 2 "Measurement_Points:Measurement_Point_Round-SMD-Pad_Big" H 5050 6225 50  0001 C CNN
-F 3 "~" H 5050 6225 50  0001 C CNN
-	1    4850 6225
-	-1   0    0    1
-$EndComp
-$Comp
-L Connector:Test_Point TP103
-U 1 1 5C0F16BF
-P 4950 6225
-F 0 "TP103" V 4950 7025 50  0000 R CNN
-F 1 "RESET_TP" V 4950 6800 50  0000 R CNN
-F 2 "Measurement_Points:Measurement_Point_Round-SMD-Pad_Big" H 5150 6225 50  0001 C CNN
-F 3 "~" H 5150 6225 50  0001 C CNN
-	1    4950 6225
-	-1   0    0    1
-$EndComp
-$Comp
-L Connector:Test_Point TP104
-U 1 1 5C0F16EB
-P 5050 6225
-F 0 "TP104" V 5050 7025 50  0000 R CNN
-F 1 "LED_0_TP" V 5050 6800 50  0000 R CNN
-F 2 "Measurement_Points:Measurement_Point_Round-SMD-Pad_Big" H 5250 6225 50  0001 C CNN
-F 3 "~" H 5250 6225 50  0001 C CNN
-	1    5050 6225
-	-1   0    0    1
-$EndComp
-$Comp
-L Connector:Test_Point TP105
-U 1 1 5C0F1719
-P 5150 6225
-F 0 "TP105" V 5150 7025 50  0000 R CNN
-F 1 "LED_1_TP" V 5150 6800 50  0000 R CNN
-F 2 "Measurement_Points:Measurement_Point_Round-SMD-Pad_Big" H 5350 6225 50  0001 C CNN
-F 3 "~" H 5350 6225 50  0001 C CNN
-	1    5150 6225
-	-1   0    0    1
-$EndComp
-$Comp
-L Connector:Test_Point TP106
-U 1 1 5C0F1747
-P 5250 6225
-F 0 "TP106" V 5250 7025 50  0000 R CNN
-F 1 "LED_2_TP" V 5250 6800 50  0000 R CNN
-F 2 "Measurement_Points:Measurement_Point_Round-SMD-Pad_Big" H 5450 6225 50  0001 C CNN
-F 3 "~" H 5450 6225 50  0001 C CNN
-	1    5250 6225
-	-1   0    0    1
-$EndComp
-$Comp
-L Connector:Test_Point TP107
-U 1 1 5C0F1773
-P 5350 6225
-F 0 "TP107" V 5350 7025 50  0000 R CNN
-F 1 "TILT_TP" V 5350 6800 50  0000 R CNN
-F 2 "Measurement_Points:Measurement_Point_Round-SMD-Pad_Big" H 5550 6225 50  0001 C CNN
-F 3 "~" H 5550 6225 50  0001 C CNN
-	1    5350 6225
-	-1   0    0    1
-$EndComp
-Wire Wire Line
-	4850 6225 4850 6050
-Wire Wire Line
-	4950 6225 4950 6050
-Wire Wire Line
-	5050 6225 5050 6050
-Wire Wire Line
-	5150 6225 5150 6050
-Wire Wire Line
-	5250 6225 5250 6050
-Wire Wire Line
-	5350 6225 5350 6050
 Wire Wire Line
 	3800 3250 4050 3250
@@
 	4050 3250 4175 3250
 Text Label 3800 3050 0    50   ~ 0
-TILT
-Text Label 5350 6050 1    50   ~ 0
 TILT
 $Comp
@@
 Wire Wire Line
 	8250 4375 8400 4375
+$Comp
+L Device:R R103
+U 1 1 5C0ECCA8
+P 7250 1025
+F 0 "R103" H 7320 1071 50  0000 L CNN
+F 1 "10k" H 7320 980 50  0000 L CNN
+F 2 "Resistors_SMD:R_0603" V 7180 1025 50  0001 C CNN
+F 3 "~" H 7250 1025 50  0001 C CNN
+	1    7250 1025
+	1    0    0    -1
+$EndComp
+$Comp
+L Device:R R102
+U 1 1 5C0ECD2E
+P 6900 1025
+F 0 "R102" H 6970 1071 50  0000 L CNN
+F 1 "10k" H 6970 980 50  0000 L CNN
+F 2 "Resistors_SMD:R_0603" V 6830 1025 50  0001 C CNN
+F 3 "~" H 6900 1025 50  0001 C CNN
+	1    6900 1025
+	1    0    0    -1
+$EndComp
+$Comp
+L power:+3V3 #PWR0109
+U 1 1 5C0ED0B8
+P 6900 875
+F 0 "#PWR0109" H 6900 725 50  0001 C CNN
+F 1 "+3V3" H 6915 1048 50  0000 C CNN
+F 2 "" H 6900 875 50  0001 C CNN
+F 3 "" H 6900 875 50  0001 C CNN
+	1    6900 875
+	1    0    0    -1
+$EndComp
+$Comp
+L power:+3V3 #PWR0137
+U 1 1 5C0ED0E1
+P 7250 875
+F 0 "#PWR0137" H 7250 725 50  0001 C CNN
+F 1 "+3V3" H 7265 1048 50  0000 C CNN
+F 2 "" H 7250 875 50  0001 C CNN
+F 3 "" H 7250 875 50  0001 C CNN
+	1    7250 875
+	1    0    0    -1
+$EndComp
+Wire Wire Line
+	6900 1400 6900 1175
+Wire Wire Line
+	6900 1400 7500 1400
+Wire Wire Line
+	6900 1400 6825 1400
+Connection ~ 6900 1400
+Wire Wire Line
+	7250 1300 7250 1175
+Wire Wire Line
+	7250 1300 7500 1300
+Wire Wire Line
+	7250 1300 7175 1300
+Connection ~ 7250 1300
 $EndSCHEMATC

Commit message: Made working tilt switch code
Connections:
- net labels removed: DEBUG
- wire segments 31 -> 27
Changed lines of the file:
@@
 Text Label 7500 3300 2    50   ~ 0
 LED_8
-Text Label 4175 3250 0    50   ~ 0
+Text Label 3800 3250 0    50   ~ 0
 LED_0
 Text Label 3800 3350 0    50   ~ 0
@@
 Wire Wire Line
 	3100 4900 3100 4950
-Text Label 4175 3150 0    50   ~ 0
-DEBUG
 $Sheet
 S 1050 1350 1350 325
@@
 	1    0    0    -1
 $EndComp
-Wire Wire Line
-	3800 3250 4050 3250
-Wire Wire Line
-	4050 3250 4050 3150
-Wire Wire Line
-	4050 3150 4175 3150
-Connection ~ 4050 3250
-Wire Wire Line
-	4050 3250 4175 3250
 Text Label 3800 3050 0    50   ~ 0
 TILT

Commit message: Began v3 board design
Parts:
- removed SW101: SW_SPST, CustomFootprints:RB-231X2, symbol Switch:SW_SPST
- added J101: Conn_02x01, Connector_PinHeader_2.54mm:PinHeader_1x02_P2.54mm_Vertical, symbol Connector_Generic:Conn_02x01
- added SW101: SW_Push, CustomFootprints:TouchButton1, symbol Switch:SW_Push
- added TP101, TP102: TestPoint, TestPoint:TestPoint_Pad_D3.0mm, symbol Connector:TestPoint
- R101: value 10k -> 976k; footprint Resistors_SMD:R_0603 -> Resistor_SMD:R_0603_1608Metric
- R102, R103: footprint Resistors_SMD:R_0603 -> Resistor_SMD:R_0603_1608Metric
Connections:
- net labels added: TOUCH
- net labels removed: TILT
- wire segments 27 -> 24
Changed lines of the file:
@@
 EESchema Schematic File Version 4
-LIBS:BalancingBusinessCardLights-cache
 EELAYER 26 0
 EELAYER END
@@
 	1    0    0    -1
 $EndComp
-Text Label 3800 3050 0    50   ~ 0
-TILT
-$Comp
-L Switch:SW_SPST SW101
-U 1 1 5C0F7A7A
-P 8050 4375
-F 0 "SW101" H 8050 4610 50  0000 C CNN
-F 1 "SW_SPST" H 8050 4519 50  0000 C CNN
-F 2 "CustomFootprints:RB-231X2" H 8050 4375 50  0001 C CNN
-F 3 "" H 8050 4375 50  0001 C CNN
-	1    8050 4375
-	1    0    0    -1
-$EndComp
-$Comp
-L Device:R R101
-U 1 1 5C0F7DAA
-P 7675 4125
-F 0 "R101" H 7745 4171 50  0000 L CNN
-F 1 "10k" H 7745 4080 50  0000 L CNN
-F 2 "Resistors_SMD:R_0603" V 7605 4125 50  0001 C CNN
-F 3 "~" H 7675 4125 50  0001 C CNN
-	1    7675 4125
-	1    0    0    -1
-$EndComp
-Text Label 7575 4375 2    50   ~ 0
-TILT
-$Comp
-L power:+3V3 #PWR0113
-U 1 1 5C0F8221
-P 7675 3975
-F 0 "#PWR0113" H 7675 3825 50  0001 C CNN
-F 1 "+3V3" H 7690 4148 50  0000 C CNN
-F 2 "" H 7675 3975 50  0001 C CNN
-F 3 "" H 7675 3975 50  0001 C CNN
-	1    7675 3975
-	1    0    0    -1
-$EndComp
-Wire Wire Line
-	7575 4375 7675 4375
-Wire Wire Line
-	7675 4375 7675 4275
-Wire Wire Line
-	7675 4375 7850 4375
-Connection ~ 7675 4375
-$Comp
-L power:GND #PWR0114
-U 1 1 5C0F8C80
-P 8400 4375
-F 0 "#PWR0114" H 8400 4125 50  0001 C CNN
-F 1 "GND" H 8405 4202 50  0000 C CNN
-F 2 "" H 8400 4375 50  0001 C CNN
-F 3 "" H 8400 4375 50  0001 C CNN
-	1    8400 4375
-	1    0    0    -1
-$EndComp
-Wire Wire Line
-	8250 4375 8400 4375
 $Comp
 L Device:R R103
@@
 F 0 "R103" H 7320 1071 50  0000 L CNN
 F 1 "10k" H 7320 980 50  0000 L CNN
-F 2 "Resistors_SMD:R_0603" V 7180 1025 50  0001 C CNN
+F 2 "Resistor_SMD:R_0603_1608Metric" V 7180 1025 50  0001 C CNN
 F 3 "~" H 7250 1025 50  0001 C CNN
 	1    7250 1025
@@
 F 0 "R102" H 6970 1071 50  0000 L CNN
 F 1 "10k" H 6970 980 50  0000 L CNN
-F 2 "Resistors_SMD:R_0603" V 6830 1025 50  0001 C CNN
+F 2 "Resistor_SMD:R_0603_1608Metric" V 6830 1025 50  0001 C CNN
 F 3 "~" H 6900 1025 50  0001 C CNN
 	1    6900 1025
@@
 	7250 1300 7175 1300
 Connection ~ 7250 1300
+$Comp
+L Connector:TestPoint TP101
+U 1 1 5C7DEA24
+P 5250 2750
+F 0 "TP101" V 5204 2938 50  0000 L CNN
+F 1 "TestPoint" V 5295 2938 50  0000 L CNN
+F 2 "TestPoint:TestPoint_Pad_D3.0mm" H 5450 2750 50  0001 C CNN
+F 3 "~" H 5450 2750 50  0001 C CNN
+	1    5250 2750
+	0    1    1    0
+$EndComp
+$Comp
+L Connector:TestPoint TP102
+U 1 1 5C7DEC98
+P 5250 2950
+F 0 "TP102" V 5204 3138 50  0000 L CNN
+F 1 "TestPoint" V 5295 3138 50  0000 L CNN
+F 2 "TestPoint:TestPoint_Pad_D3.0mm" H 5450 2950 50  0001 C CNN
+F 3 "~" H 5450 2950 50  0001 C CNN
+	1    5250 2950
+	0    1    1    0
+$EndComp
+Text Label 5250 2750 2    50   ~ 0
+SDA
+Text Label 5250 2950 2    50   ~ 0
+SCL
+$Comp
+L Connector_Generic:Conn_02x01 J101
+U 1 1 5C7DF1A3
+P 5400 3450
+F 0 "J101" H 5450 3667 50  0000 C CNN
+F 1 "Conn_02x01" H 5450 3576 50  0000 C CNN
+F 2 "Connector_PinHeader_2.54mm:PinHeader_1x02_P2.54mm_Vertical" H 5400 3450 50  0001 C CNN
+F 3 "~" H 5400 3450 50  0001 C CNN
+	1    5400 3450
+	1    0    0    -1
+$EndComp
+$Comp
+L power:+3V3 #PWR0106
+U 1 1 5C7DF23F
+P 5700 3450
+F 0 "#PWR0106" H 5700 3300 50  0001 C CNN
+F 1 "+3V3" H 5715 3623 50  0000 C CNN
+F 2 "" H 5700 3450 50  0001 C CNN
+F 3 "" H 5700 3450 50  0001 C CNN
+	1    5700 3450
+	0    1    1    0
+$EndComp
+$Comp
+L power:GND #PWR0111
+U 1 1 5C7DF2BD
+P 5200 3450
+F 0 "#PWR0111" H 5200 3200 50  0001 C CNN
+F 1 "GND" H 5205 3277 50  0000 C CNN
+F 2 "" H 5200 3450 50  0001 C CNN
+F 3 "" H 5200 3450 50  0001 C CNN
+	1    5200 3450
+	1    0    0    -1
+$EndComp
+$Comp
+L Switch:SW_Push SW101
+U 1 1 5C7E16C0
+P 8200 4300
+F 0 "SW101" H 8200 4585 50  0000 C CNN
+F 1 "SW_Push" H 8200 4494 50  0000 C CNN
+F 2 "CustomFootprints:TouchButton1" H 8200 4500 50  0001 C CNN
+F 3 "" H 8200 4500 50  0001 C CNN
+	1    8200 4300
+	1    0    0    -1
+$EndComp
+$Comp
+L power:GND #PWR0114
+U 1 1 5C7E1777
+P 8400 4300
+F 0 "#PWR0114" H 8400 4050 50  0001 C CNN
+F 1 "GND" H 8405 4127 50  0000 C CNN
+F 2 "" H 8400 4300 50  0001 C CNN
+F 3 "" H 8400 4300 50  0001 C CNN
+	1    8400 4300
+	1    0    0    -1
+$EndComp
+$Comp
+L power:+3V3 #PWR0113
+U 1 1 5C7E1803
+P 7600 4300
+F 0 "#PWR0113" H 7600 4150 50  0001 C CNN
+F 1 "+3V3" V 7615 4428 50  0000 L CNN
+F 2 "" H 7600 4300 50  0001 C CNN
+F 3 "" H 7600 4300 50  0001 C CNN
+	1    7600 4300
+	0    -1   -1   0
+$EndComp
+Text Label 8000 4300 1    50   ~ 0
+TOUCH
+$Comp
+L Device:R R101
+U 1 1 5C7E1882
+P 7750 4300
+F 0 "R101" V 7543 4300 50  0000 C CNN
+F 1 "976k" V 7634 4300 50  0000 C CNN
+F 2 "Resistor_SMD:R_0603_1608Metric" V 7680 4300 50  0001 C CNN
+F 3 "~" H 7750 4300 50  0001 C CNN
+	1    7750 4300
+	0    1    1    0
+$EndComp
+Wire Wire Line
+	7900 4300 8000 4300
+Text Label 3800 3050 0    50   ~ 0
+TOUCH
 $EndSCHEMATC

Commit message: Right Stuff
Parts:
- removed SW101: SW_Push, CustomFootprints:TouchButton1, symbol Switch:SW_Push
- added BTN?: Cap Sense, symbol Connector:Test_Point
- added C?: 22pf, symbol Device:C
- TP101, TP102: symbol Connector:TestPoint -> Connector:Test_Point
Connections:
- net labels added: TOUCH_RECEIVE, TOUCH_REVEIVE, TOUCH_SEND
- net labels removed: TOUCH
- wire segments 24 -> 26
Changed lines of the file:
@@
 	1    0    0    -1
 $EndComp
-Text Label 4100 3850 0    50   ~ 0
+Text Label 4900 3850 0    50   ~ 0
 MOSI
 Text Label 4100 3950 0    50   ~ 0
@@
 $EndComp
 Wire Wire Line
-	3800 3850 4100 3850
-Wire Wire Line
 	3800 4050 4100 4050
 Wire Wire Line
@@
 Connection ~ 7250 1300
 $Comp
-L Connector:TestPoint TP101
+L Connector:Test_Point TP101
 U 1 1 5C7DEA24
 P 5250 2750
@@
 $EndComp
 $Comp
-L Connector:TestPoint TP102
+L Connector:Test_Point TP102
 U 1 1 5C7DEC98
 P 5250 2950
@@
 $EndComp
 $Comp
-L Switch:SW_Push SW101
-U 1 1 5C7E16C0
-P 8200 4300
-F 0 "SW101" H 8200 4585 50  0000 C CNN
-F 1 "SW_Push" H 8200 4494 50  0000 C CNN
-F 2 "CustomFootprints:TouchButton1" H 8200 4500 50  0001 C CNN
-F 3 "" H 8200 4500 50  0001 C CNN
-	1    8200 4300
-	1    0    0    -1
-$EndComp
-$Comp
 L power:GND #PWR0114
 U 1 1 5C7E1777
-P 8400 4300
-F 0 "#PWR0114" H 8400 4050 50  0001 C CNN
-F 1 "GND" H 8405 4127 50  0000 C CNN
-F 2 "" H 8400 4300 50  0001 C CNN
-F 3 "" H 8400 4300 50  0001 C CNN
-	1    8400 4300
-	1    0    0    -1
-$EndComp
-$Comp
-L power:+3V3 #PWR0113
-U 1 1 5C7E1803
-P 7600 4300
-F 0 "#PWR0113" H 7600 4150 50  0001 C CNN
-F 1 "+3V3" V 7615 4428 50  0000 L CNN
-F 2 "" H 7600 4300 50  0001 C CNN
-F 3 "" H 7600 4300 50  0001 C CNN
-	1    7600 4300
-	0    -1   -1   0
+P 8000 4600
+F 0 "#PWR0114" H 8000 4350 50  0001 C CNN
+F 1 "GND" H 8005 4427 50  0000 C CNN
+F 2 "" H 8000 4600 50  0001 C CNN
+F 3 "" H 8000 4600 50  0001 C CNN
+	1    8000 4600
+	1    0    0    -1
 $EndComp
 Text Label 8000 4300 1    50   ~ 0
-TOUCH
+TOUCH_REVEIVE
 $Comp
 L Device:R R101
@@
 	0    1    1    0
 $EndComp
+Text Label 4400 3850 1    50   ~ 0
+TOUCH_SEND
+Text Label 3800 3050 0    50   ~ 0
+TOUCH_RECEIVE
+Wire Wire Line
+	3800 3850 4900 3850
+Text Label 7325 4300 2    50   ~ 0
+TOUCH_SEND
+Wire Wire Line
+	7325 4300 7600 4300
+$Comp
+L Device:C C?
+U 1 1 5C837217
+P 8000 4450
+F 0 "C?" H 8115 4496 50  0000 L CNN
+F 1 "22pf" H 8115 4405 50  0000 L CNN
+F 2 "" H 8038 4300 50  0001 C CNN
+F 3 "~" H 8000 4450 50  0001 C CNN
+	1    8000 4450
+	1    0    0    -1
+$EndComp
+$Comp
+L Connector:Test_Point BTN?
+U 1 1 5C837578
+P 8400 4300
+F 0 "BTN?" H 8458 4420 50  0000 L CNN
+F 1 "Cap Sense" H 8458 4329 50  0000 L CNN
+F 2 "" H 8600 4300 50  0001 C CNN
+F 3 "~" H 8600 4300 50  0001 C CNN
+	1    8400 4300
+	1    0    0    -1
+$EndComp
 Wire Wire Line
 	7900 4300 8000 4300
-Text Label 3800 3050 0    50   ~ 0
-TOUCH
+Connection ~ 8000 4300
+Wire Wire Line
+	8000 4300 8400 4300
 $EndSCHEMATC

Commit message: Made touch sense cap
Parts:
- BTN?: footprint (none) -> CustomFootprints:CAP_TOUCH
- C?: footprint (none) -> Capacitors_SMD:C_0603
Changed lines of the file:
@@
 EESchema Schematic File Version 4
+LIBS:BalancingBusinessCardLights-cache
 EELAYER 26 0
 EELAYER END
@@
 F 0 "C?" H 8115 4496 50  0000 L CNN
 F 1 "22pf" H 8115 4405 50  0000 L CNN
-F 2 "" H 8038 4300 50  0001 C CNN
+F 2 "Capacitors_SMD:C_0603" H 8038 4300 50  0001 C CNN
 F 3 "~" H 8000 4450 50  0001 C CNN
 	1    8000 4450
@@
 F 0 "BTN?" H 8458 4420 50  0000 L CNN
 F 1 "Cap Sense" H 8458 4329 50  0000 L CNN
-F 2 "" H 8600 4300 50  0001 C CNN
+F 2 "CustomFootprints:CAP_TOUCH" H 8600 4300 50  0001 C CNN
 F 3 "~" H 8600 4300 50  0001 C CNN
 	1    8400 4300

Commit message: Made custom test point symbol
Parts:
- BTN?, TP101, TP102: symbol Connector:Test_Point -> Custom:Test_Point
Changed lines of the file:
@@
 Connection ~ 7250 1300
 $Comp
-L Connector:Test_Point TP101
+L Custom:Test_Point TP101
 U 1 1 5C7DEA24
 P 5250 2750
@@
 $EndComp
 $Comp
-L Connector:Test_Point TP102
+L Custom:Test_Point TP102
 U 1 1 5C7DEC98
 P 5250 2950
@@
 $EndComp
 $Comp
-L Connector:Test_Point BTN?
+L Custom:Test_Point BTN?
 U 1 1 5C837578
 P 8400 4300

Commit message: Got a better test point
Parts:
- TP101, TP102: footprint TestPoint:TestPoint_Pad_D3.0mm -> Measurement_Points:Measurement_Point_Round-SMD-Pad_Small
Changed lines of the file:
@@
 F 0 "TP101" V 5204 2938 50  0000 L CNN
 F 1 "TestPoint" V 5295 2938 50  0000 L CNN
-F 2 "TestPoint:TestPoint_Pad_D3.0mm" H 5450 2750 50  0001 C CNN
+F 2 "Measurement_Points:Measurement_Point_Round-SMD-Pad_Small" H 5450 2750 50  0001 C CNN
 F 3 "~" H 5450 2750 50  0001 C CNN
 	1    5250 2750
@@
 F 0 "TP102" V 5204 3138 50  0000 L CNN
 F 1 "TestPoint" V 5295 3138 50  0000 L CNN
-F 2 "TestPoint:TestPoint_Pad_D3.0mm" H 5450 2950 50  0001 C CNN
+F 2 "Measurement_Points:Measurement_Point_Round-SMD-Pad_Small" H 5450 2950 50  0001 C CNN
 F 3 "~" H 5450 2950 50  0001 C CNN
 	1    5250 2950
