File: Design/BalancingBusinessCard/BalancingBusinessCardLights.sch (KiCad schematic (older format))
At the start: 12 parts, among them J101 Conn_02x01, U101 ATtiny261A-MU

Commit message: Cleaned up fills
Parts:
- C2: renamed from C?; footprint Capacitors_SMD:C_0603 -> Capacitor_SMD:C_0603_1608Metric
- TP1: renamed from TP101; footprint Measurement_Points:Measurement_Point_Round-SMD-Pad_Small -> TestPoint:TestPoint_Pad_D1.0mm
- TP2: renamed from TP102; footprint Measurement_Points:Measurement_Point_Round-SMD-Pad_Small -> TestPoint:TestPoint_Pad_D1.0mm
- gave numbers to parts that had none: 1
- renumbered BT101 to BT1, C101 to C1, J101 to J1, R102 to R1, R103 to R2, R101 to R3, U101 to U1
Connections:
- net labels removed: TOUCH_REVEIVE
Changed lines of the file:
@@
 SCL
 $Comp
-L Device:Battery BT101
+L Device:Battery BT1
 U 1 1 5BCBEFF8
 P 4400 1300
-F 0 "BT101" H 4508 1346 50  0000 L CNN
+F 0 "BT1" H 4508 1346 50  0000 L CNN
 F 1 "Battery" H 4508 1255 50  0000 L CNN
 F 2 "CustomFootprints:CR2016VP" V 4400 1360 50  0001 C CNN
@@
 $EndComp
 $Comp
-L power:+BATT #PWR0101
+L power:+BATT #PWR09
 U 1 1 5BCBF44A
 P 4400 1050
-F 0 "#PWR0101" H 4400 900 50  0001 C CNN
+F 0 "#PWR09" H 4400 900 50  0001 C CNN
 F 1 "+BATT" H 4415 1223 50  0000 C CNN
 F 2 "" H 4400 1050 50  0001 C CNN
@@
 +3V
 $Comp
-L power:GND #PWR0102
+L power:GND #PWR010
 U 1 1 5BCBF4A9
 P 4400 1500
-F 0 "#PWR0102" H 4400 1250 50  0001 C CNN
+F 0 "#PWR010" H 4400 1250 50  0001 C CNN
 F 1 "GND" H 4405 1327 50  0000 C CNN
 F 2 "" H 4400 1500 50  0001 C CNN
@@
 MOSI
 $Comp
-L power:GND #PWR0107
+L power:GND #PWR06
 U 1 1 5BCBF839
 P 3300 5950
-F 0 "#PWR0107" H 3300 5700 50  0001 C CNN
+F 0 "#PWR06" H 3300 5700 50  0001 C CNN
 F 1 "GND" V 3305 5822 50  0000 R CNN
 F 2 "" H 3300 5950 50  0001 C CNN
@@
 RESET
 $Comp
-L power:GND #PWR0108
+L power:GND #PWR04
 U 1 1 5BCCA97D
 P 3100 4950
-F 0 "#PWR0108" H 3100 4700 50  0001 C CNN
+F 0 "#PWR04" H 3100 4700 50  0001 C CNN
 F 1 "GND" H 3105 4777 50  0000 C CNN
 F 2 "" H 3100 4950 50  0001 C CNN
@@
 	3100 2400 3450 2400
 $Comp
-L Device:C C101
+L Device:C C1
 U 1 1 5BCC392A
 P 3600 2400
-F 0 "C101" V 3852 2400 50  0000 C CNN
+F 0 "C1" V 3852 2400 50  0000 C CNN
 F 1 "10uF" V 3761 2400 50  0000 C CNN
 F 2 "Capacitor_SMD:C_0805_2012Metric" H 3638 2250 50  0001 C CNN
@@
 $EndComp
 $Comp
-L power:GND #PWR0112
+L power:GND #PWR07
 U 1 1 5BCC3A23
 P 3750 2400
-F 0 "#PWR0112" H 3750 2150 50  0001 C CNN
+F 0 "#PWR07" H 3750 2150 50  0001 C CNN
 F 1 "GND" H 3755 2227 50  0000 C CNN
 F 2 "" H 3750 2400 50  0001 C CNN
@@
 	3800 3950 4100 3950
 $Comp
-L power:PWR_FLAG #FLG0101
+L power:PWR_FLAG #FLG01
 U 1 1 5BCC0D87
 P 4050 1100
-F 0 "#FLG0101" H 4050 1175 50  0001 C CNN
+F 0 "#FLG01" H 4050 1175 50  0001 C CNN
 F 1 "PWR_FLAG" H 4050 1274 50  0000 C CNN
 F 2 "" H 4050 1100 50  0001 C CNN
@@
 	4050 1100 4400 1100
 $Comp
-L power:PWR_FLAG #FLG0102
+L power:PWR_FLAG #FLG02
 U 1 1 5BCC114E
 P 4050 1400
-F 0 "#FLG0102" H 4050 1475 50  0001 C CNN
+F 0 "#FLG02" H 4050 1475 50  0001 C CNN
 F 1 "PWR_FLAG" H 4050 1574 50  0000 C CNN
 F 2 "" H 4050 1400 50  0001 C CNN
@@
 	4050 1450 4050 1400
 $Comp
-L power:GND #PWR0134
+L power:GND #PWR08
 U 1 1 5BCC13FA
 P 4050 1450
-F 0 "#PWR0134" H 4050 1200 50  0001 C CNN
+F 0 "#PWR08" H 4050 1200 50  0001 C CNN
 F 1 "GND" H 4055 1277 50  0000 C CNN
 F 2 "" H 4050 1450 50  0001 C CNN
@@
 $EndComp
 $Comp
-L MCU_Microchip_ATtiny:ATtiny261A-MU U101
+L MCU_Microchip_ATtiny:ATtiny261A-MU U1
 U 1 1 5C0B1B62
 P 3100 3750
-F 0 "U101" H 2459 3796 50  0000 R CNN
+F 0 "U1" H 2459 3796 50  0000 R CNN
 F 1 "ATtiny261A-MU" H 2459 3705 50  0000 R CNN
 F 2 "Housings_DFN_QFN:QFN-32-1EP_5x5mm_Pitch0.5mm" H 3100 3750 50  0001 C CIN
@@
 $EndSheet
 $Comp
-L power:+3V3 #PWR0103
+L power:+3V3 #PWR02
 U 1 1 5C0EE9D9
 P 2750 1550
-F 0 "#PWR0103" H 2750 1400 50  0001 C CNN
+F 0 "#PWR02" H 2750 1400 50  0001 C CNN
 F 1 "+3V3" H 2765 1723 50  0000 C CNN
 F 2 "" H 2750 1550 50  0001 C CNN
@@
 	2400 1550 2750 1550
 $Comp
-L power:+BATT #PWR0104
+L power:+BATT #PWR01
 U 1 1 5C0EEBFA
 P 2525 1425
-F 0 "#PWR0104" H 2525 1275 50  0001 C CNN
+F 0 "#PWR01" H 2525 1275 50  0001 C CNN
 F 1 "+BATT" H 2540 1598 50  0000 C CNN
 F 2 "" H 2525 1425 50  0001 C CNN
@@
 	2400 1425 2525 1425
 $Comp
-L power:+3V3 #PWR0105
+L power:+3V3 #PWR03
 U 1 1 5C0EF8B9
 P 3100 2400
-F 0 "#PWR0105" H 3100 2250 50  0001 C CNN
+F 0 "#PWR03" H 3100 2250 50  0001 C CNN
 F 1 "+3V3" H 3115 2573 50  0000 C CNN
 F 2 "" H 3100 2400 50  0001 C CNN
@@
 Connection ~ 3100 2400
 $Comp
-L power:+3V3 #PWR0110
+L power:+3V3 #PWR05
 U 1 1 5C0EF953
 P 3300 5750
-F 0 "#PWR0110" H 3300 5600 50  0001 C CNN
+F 0 "#PWR05" H 3300 5600 50  0001 C CNN
 F 1 "+3V3" H 3315 5923 50  0000 C CNN
 F 2 "" H 3300 5750 50  0001 C CNN
@@
 $EndComp
 $Comp
-L Device:R R103
+L Device:R R2
 U 1 1 5C0ECCA8
 P 7250 1025
-F 0 "R103" H 7320 1071 50  0000 L CNN
+F 0 "R2" H 7320 1071 50  0000 L CNN
 F 1 "10k" H 7320 980 50  0000 L CNN
 F 2 "Resistor_SMD:R_0603_1608Metric" V 7180 1025 50  0001 C CNN
@@
 $EndComp
 $Comp
-L Device:R R102
+L Device:R R1
 U 1 1 5C0ECD2E
 P 6900 1025
-F 0 "R102" H 6970 1071 50  0000 L CNN
+F 0 "R1" H 6970 1071 50  0000 L CNN
 F 1 "10k" H 6970 980 50  0000 L CNN
 F 2 "Resistor_SMD:R_0603_1608Metric" V 6830 1025 50  0001 C CNN
@@
 $EndComp
 $Comp
-L power:+3V3 #PWR0109
+L power:+3V3 #PWR013
 U 1 1 5C0ED0B8
 P 6900 875
-F 0 "#PWR0109" H 6900 725 50  0001 C CNN
+F 0 "#PWR013" H 6900 725 50  0001 C CNN
 F 1 "+3V3" H 6915 1048 50  0000 C CNN
 F 2 "" H 6900 875 50  0001 C CNN
@@
 $EndComp
 $Comp
-L power:+3V3 #PWR0137
+L power:+3V3 #PWR014
 U 1 1 5C0ED0E1
 P 7250 875
-F 0 "#PWR0137" H 7250 725 50  0001 C CNN
+F 0 "#PWR014" H 7250 725 50  0001 C CNN
 F 1 "+3V3" H 7265 1048 50  0000 C CNN
 F 2 "" H 7250 875 50  0001 C CNN
@@
 Connection ~ 7250 1300
 $Comp
-L Custom:Test_Point TP101
+L Custom:Test_Point TP1
 U 1 1 5C7DEA24
 P 5250 2750
-F 0 "TP101" V 5204 2938 50  0000 L CNN
+F 0 "TP1" V 5204 2938 50  0000 L CNN
 F 1 "TestPoint" V 5295 2938 50  0000 L CNN
-F 2 "Measurement_Points:Measurement_Point_Round-SMD-Pad_Small" H 5450 2750 50  0001 C CNN
+F 2 "TestPoint:TestPoint_Pad_D1.0mm" H 5450 2750 50  0001 C CNN
 F 3 "~" H 5450 2750 50  0001 C CNN
 	1    5250 2750
@@
 $EndComp
 $Comp
-L Custom:Test_Point TP102
+L Custom:Test_Point TP2
 U 1 1 5C7DEC98
 P 5250 2950
-F 0 "TP102" V 5204 3138 50  0000 L CNN
+F 0 "TP2" V 5204 3138 50  0000 L CNN
 F 1 "TestPoint" V 5295 3138 50  0000 L CNN
-F 2 "Measurement_Points:Measurement_Point_Round-SMD-Pad_Small" H 5450 2950 50  0001 C CNN
+F 2 "TestPoint:TestPoint_Pad_D1.0mm" H 5450 2950 50  0001 C CNN
 F 3 "~" H 5450 2950 50  0001 C CNN
 	1    5250 2950
@@
 SCL
 $Comp
-L Connector_Generic:Conn_02x01 J101
+L Connector_Generic:Conn_02x01 J1
 U 1 1 5C7DF1A3
 P 5400 3450
-F 0 "J101" H 5450 3667 50  0000 C CNN
+F 0 "J1" H 5450 3667 50  0000 C CNN
 F 1 "Conn_02x01" H 5450 3576 50  0000 C CNN
 F 2 "Connector_PinHeader_2.54mm:PinHeader_1x02_P2.54mm_Vertical" H 5400 3450 50  0001 C CNN
@@
 $EndComp
 $Comp
-L power:+3V3 #PWR0106
+L power:+3V3 #PWR012
 U 1 1 5C7DF23F
 P 5700 3450
-F 0 "#PWR0106" H 5700 3300 50  0001 C CNN
+F 0 "#PWR012" H 5700 3300 50  0001 C CNN
 F 1 "+3V3" H 5715 3623 50  0000 C CNN
 F 2 "" H 5700 3450 50  0001 C CNN
@@
 $EndComp
 $Comp
-L power:GND #PWR0111
+L power:GND #PWR011
 U 1 1 5C7DF2BD
 P 5200 3450
-F 0 "#PWR0111" H 5200 3200 50  0001 C CNN
+F 0 "#PWR011" H 5200 3200 50  0001 C CNN
 F 1 "GND" H 5205 3277 50  0000 C CNN
 F 2 "" H 5200 3450 50  0001 C CNN
@@
 $EndComp
 $Comp
-L power:GND #PWR0114
+L power:GND #PWR015
 U 1 1 5C7E1777
 P 8000 4600
-F 0 "#PWR0114" H 8000 4350 50  0001 C CNN
+F 0 "#PWR015" H 8000 4350 50  0001 C CNN
 F 1 "GND" H 8005 4427 50  0000 C CNN
 F 2 "" H 8000 4600 50  0001 C CNN
@@
 $EndComp
 Text Label 8000 4300 1    50   ~ 0
-TOUCH_REVEIVE
-$Comp
-L Device:R R101
+TOUCH_RECEIVE
+$Comp
+L Device:R R3
 U 1 1 5C7E1882
 P 7750 4300
-F 0 "R101" V 7543 4300 50  0000 C CNN
+F 0 "R3" V 7543 4300 50  0000 C CNN
 F 1 "976k" V 7634 4300 50  0000 C CNN
 F 2 "Resistor_SMD:R_0603_1608Metric" V 7680 4300 50  0001 C CNN
@@
 	7325 4300 7600 4300
 $Comp
-L Device:C C?
+L Device:C C2
 U 1 1 5C837217
 P 8000 4450
-F 0 "C?" H 8115 4496 50  0000 L CNN
+F 0 "C2" H 8115 4496 50  0000 L CNN
 F 1 "22pf" H 8115 4405 50  0000 L CNN
-F 2 "Capacitors_SMD:C_0603" H 8038 4300 50  0001 C CNN
+F 2 "Capacitor_SMD:C_0603_1608Metric" H 8038 4300 50  0001 C CNN
 F 3 "~" H 8000 4450 50  0001 C CNN
 	1    8000 4450
@@
 $EndComp
 $Comp
-L Custom:Test_Point BTN?
+L Custom:Test_Point BTN1
 U 1 1 5C837578
 P 8400 4300
-F 0 "BTN?" H 8458 4420 50  0000 L CNN
+F 0 "BTN1" H 8458 4420 50  0000 L CNN
 F 1 "Cap Sense" H 8458 4329 50  0000 L CNN
 F 2 "CustomFootprints:CAP_TOUCH" H 8600 4300 50  0001 C CNN
