File: Design/BalancingBusinessCard/BalancingBusinessCardLights.sch (KiCad schematic (older format))
At the start: 12 parts, among them J1 Conn_02x01, U1 ATtiny261A-MU

Commit message: Updated names
Parts:
- BT1: value Battery -> CR-2016
- ICSP1: value Conn_02x03_Odd_Even -> ICSP
- J1: value Conn_02x01 -> PWR
- U1: value ATtiny261A-MU -> ATTINY861-15MZ
Changed lines of the file:
@@
 EESchema Schematic File Version 4
 LIBS:BalancingBusinessCardLights-cache
-EELAYER 26 0
+EELAYER 29 0
 EELAYER END
 $Descr A4 11693 8268
@@
 P 4400 1300
 F 0 "BT1" H 4508 1346 50  0000 L CNN
-F 1 "Battery" H 4508 1255 50  0000 L CNN
+F 1 "CR-2016" H 4508 1255 50  0000 L CNN
 F 2 "CustomFootprints:CR2016VP" V 4400 1360 50  0001 C CNN
 F 3 "~" V 4400 1360 50  0001 C CNN
@@
 P 3000 5850
 F 0 "ICSP1" H 3050 6050 50  0000 C CNN
-F 1 "Conn_02x03_Odd_Even" H 3050 5650 50  0000 C CNN
+F 1 "ICSP" H 3050 5650 50  0000 C CNN
 F 2 "Connector_PinHeader_2.54mm:PinHeader_2x03_P2.54mm_Vertical" H 3000 5850 50  0001 C CNN
 F 3 "~" H 3000 5850 50  0001 C CNN
@@
 P 3100 3750
 F 0 "U1" H 2459 3796 50  0000 R CNN
-F 1 "ATtiny261A-MU" H 2459 3705 50  0000 R CNN
+F 1 "ATTINY861-15MZ" H 2459 3705 50  0000 R CNN
 F 2 "Housings_DFN_QFN:QFN-32-1EP_5x5mm_Pitch0.5mm" H 3100 3750 50  0001 C CIN
 F 3 "http://ww1.microchip.com/downloads/en/DeviceDoc/doc8197.pdf" H 3100 3750 50  0001 C CNN
@@
 P 5400 3450
 F 0 "J1" H 5450 3667 50  0000 C CNN
-F 1 "Conn_02x01" H 5450 3576 50  0000 C CNN
+F 1 "PWR" H 5450 3576 50  0000 C CNN
 F 2 "Connector_PinHeader_2.54mm:PinHeader_1x02_P2.54mm_Vertical" H 5400 3450 50  0001 C CNN
 F 3 "~" H 5400 3450 50  0001 C CNN
