File: Design/BalancingBusinessCard/3V3Regulator.sch (KiCad schematic (older format))
At the start: 6 parts, among them U402 MCP1640DCH

Commit message: Finished light board layout and silkscreen design
Parts:
- U402: footprint Package_TO_SOT_SMD:SOT-23-6 -> TO_SOT_Packages_SMD:SOT-23-6
Changed lines of the file:
@@
 F 0 "U402" H 2825 2642 50  0000 C CNN
 F 1 "MCP1640DCH" H 2825 2551 50  0000 C CNN
-F 2 "Package_TO_SOT_SMD:SOT-23-6" H 2875 1925 50  0001 L CIN
+F 2 "TO_SOT_Packages_SMD:SOT-23-6" H 2875 1925 50  0001 L CIN
 F 3 "http://ww1.microchip.com/downloads/en/DeviceDoc/20002234D.pdf" H 2575 2625 50  0001 C CNN
 	1    2825 2175

Commit message: Made working tilt switch code
Parts:
- C404: footprint Capacitors_SMD:C_0603 -> Capacitors_SMD:C_0805
Changed lines of the file:
@@
 F 0 "C404" H 4115 2271 50  0000 L CNN
 F 1 "10uF" H 4115 2180 50  0000 L CNN
-F 2 "Capacitors_SMD:C_0603" H 4038 2075 50  0001 C CNN
+F 2 "Capacitors_SMD:C_0805" H 4038 2075 50  0001 C CNN
 F 3 "~" H 4000 2225 50  0001 C CNN
 	1    4000 2225

Commit message: Began v3 board design
Parts:
- C404: footprint Capacitors_SMD:C_0805 -> Capacitor_SMD:C_0805_2012Metric
- R401, R402: footprint Resistors_SMD:R_0603 -> Resistor_SMD:R_0603_1608Metric
Changed lines of the file:
@@
 EESchema Schematic File Version 4
-LIBS:BalancingBusinessCardLights-cache
 EELAYER 26 0
 EELAYER END
@@
 F 0 "R401" H 3595 2271 50  0000 L CNN
 F 1 "976k" H 3595 2180 50  0000 L CNN
-F 2 "Resistors_SMD:R_0603" V 3455 2225 50  0001 C CNN
+F 2 "Resistor_SMD:R_0603_1608Metric" V 3455 2225 50  0001 C CNN
 F 3 "~" H 3525 2225 50  0001 C CNN
 	1    3525 2225
@@
 F 0 "R402" H 3595 2621 50  0000 L CNN
 F 1 "562k" H 3595 2530 50  0000 L CNN
-F 2 "Resistors_SMD:R_0603" V 3455 2575 50  0001 C CNN
+F 2 "Resistor_SMD:R_0603_1608Metric" V 3455 2575 50  0001 C CNN
 F 3 "~" H 3525 2575 50  0001 C CNN
 	1    3525 2575
@@
 F 0 "C404" H 4115 2271 50  0000 L CNN
 F 1 "10uF" H 4115 2180 50  0000 L CNN
-F 2 "Capacitors_SMD:C_0805" H 4038 2075 50  0001 C CNN
+F 2 "Capacitor_SMD:C_0805_2012Metric" H 4038 2075 50  0001 C CNN
 F 3 "~" H 4000 2225 50  0001 C CNN
 	1    4000 2225

Commit message: Cleaned up fills
Parts:
- C5: renamed from C403; footprint Capacitors_SMD:C_0603 -> Capacitor_SMD:C_0603_1608Metric
- renumbered C404 to C6, L401 to L1, R401 to R13, R402 to R14, U402 to U3
Changed lines of the file:
@@
 $EndDescr
 $Comp
-L Regulator_Switching:MCP1640DCH U402
+L Regulator_Switching:MCP1640DCH U3
 U 1 1 5C0ED17A
 P 2825 2175
-F 0 "U402" H 2825 2642 50  0000 C CNN
+F 0 "U3" H 2825 2642 50  0000 C CNN
 F 1 "MCP1640DCH" H 2825 2551 50  0000 C CNN
 F 2 "TO_SOT_Packages_SMD:SOT-23-6" H 2875 1925 50  0001 L CIN
@@
 $EndComp
 $Comp
-L Device:C C403
+L Device:C C5
 U 1 1 5C0ED297
 P 2050 2125
-F 0 "C403" H 2165 2171 50  0000 L CNN
+F 0 "C5" H 2165 2171 50  0000 L CNN
 F 1 "4.7uF" H 2165 2080 50  0000 L CNN
-F 2 "Capacitors_SMD:C_0603" H 2088 1975 50  0001 C CNN
+F 2 "Capacitor_SMD:C_0603_1608Metric" H 2088 1975 50  0001 C CNN
 F 3 "~" H 2050 2125 50  0001 C CNN
 	1    2050 2125
@@
 $EndComp
 $Comp
-L Device:L L401
+L Device:L L1
 U 1 1 5C0ED346
 P 2825 1550
-F 0 "L401" V 2647 1550 50  0000 C CNN
+F 0 "L1" V 2647 1550 50  0000 C CNN
 F 1 "4.7uH" V 2738 1550 50  0000 C CNN
 F 2 "Inductors_SMD:L_0603" H 2825 1550 50  0001 C CNN
@@
 	2350 1975 2050 1975
 $Comp
-L power:GND #PWR0115
+L power:GND #PWR033
 U 1 1 5C0ED540
 P 2050 2275
-F 0 "#PWR0115" H 2050 2025 50  0001 C CNN
+F 0 "#PWR033" H 2050 2025 50  0001 C CNN
 F 1 "GND" H 2055 2102 50  0000 C CNN
 F 2 "" H 2050 2275 50  0001 C CNN
@@
 $EndComp
 $Comp
-L power:GND #PWR0116
+L power:GND #PWR034
 U 1 1 5C0ED558
 P 2825 2475
-F 0 "#PWR0116" H 2825 2225 50  0001 C CNN
+F 0 "#PWR034" H 2825 2225 50  0001 C CNN
 F 1 "GND" H 2830 2302 50  0000 C CNN
 F 2 "" H 2825 2475 50  0001 C CNN
@@
 $EndComp
 $Comp
-L power:GND #PWR0126
+L power:GND #PWR035
 U 1 1 5C0ED5C1
 P 3525 2775
-F 0 "#PWR0126" H 3525 2525 50  0001 C CNN
+F 0 "#PWR035" H 3525 2525 50  0001 C CNN
 F 1 "GND" H 3530 2602 50  0000 C CNN
 F 2 "" H 3525 2775 50  0001 C CNN
@@
 	3300 1975 3225 1975
 $Comp
-L Device:R R401
+L Device:R R13
 U 1 1 5C0ED6C5
 P 3525 2225
-F 0 "R401" H 3595 2271 50  0000 L CNN
+F 0 "R13" H 3595 2271 50  0000 L CNN
 F 1 "976k" H 3595 2180 50  0000 L CNN
 F 2 "Resistor_SMD:R_0603_1608Metric" V 3455 2225 50  0001 C CNN
@@
 $EndComp
 $Comp
-L Device:R R402
+L Device:R R14
 U 1 1 5C0ED701
 P 3525 2575
-F 0 "R402" H 3595 2621 50  0000 L CNN
+F 0 "R14" H 3595 2621 50  0000 L CNN
 F 1 "562k" H 3595 2530 50  0000 L CNN
 F 2 "Resistor_SMD:R_0603_1608Metric" V 3455 2575 50  0001 C CNN
@@
 	3525 2775 3525 2725
 $Comp
-L Device:C C404
+L Device:C C6
 U 1 1 5C0EDB53
 P 4000 2225
-F 0 "C404" H 4115 2271 50  0000 L CNN
+F 0 "C6" H 4115 2271 50  0000 L CNN
 F 1 "10uF" H 4115 2180 50  0000 L CNN
 F 2 "Capacitor_SMD:C_0805_2012Metric" H 4038 2075 50  0001 C CNN
@@
 $EndComp
 $Comp
-L power:GND #PWR0135
+L power:GND #PWR036
 U 1 1 5C0EDC94
 P 4000 2425
-F 0 "#PWR0135" H 4000 2175 50  0001 C CNN
+F 0 "#PWR036" H 4000 2175 50  0001 C CNN
 F 1 "GND" H 4005 2252 50  0000 C CNN
 F 2 "" H 4000 2425 50  0001 C CNN

Commit message: Updated names
Parts:
- U3: value MCP1640DCH -> MCP1640DT-I/CHY
Changed lines of the file:
@@
 EESchema Schematic File Version 4
 LIBS:BalancingBusinessCardLights-cache
-EELAYER 26 0
+EELAYER 29 0
 EELAYER END
 $Descr A4 11693 8268
@@
 P 2825 2175
 F 0 "U3" H 2825 2642 50  0000 C CNN
-F 1 "MCP1640DCH" H 2825 2551 50  0000 C CNN
+F 1 "MCP1640DT-I/CHY" H 2825 2551 50  0000 C CNN
 F 2 "TO_SOT_Packages_SMD:SOT-23-6" H 2875 1925 50  0001 L CIN
 F 3 "http://ww1.microchip.com/downloads/en/DeviceDoc/20002234D.pdf" H 2575 2625 50  0001 C CNN
