File: design/business_card/business_card.kicad_pcb (KiCad board)
At the start: 2 copper layers, 54 x 86 mm, 34 parts, among them U101 ATtiny861A-M, U102 ST25TA02KB-DC6H5, U103 LIS3DHTR

Commit message: Routing complete
Parts:
- added L101: 2.75uH, CustomFootprints:Trace_Inductor_2_75uH, F.Cu at (225.4, 65.2)
- U102: value ST25TA02KB-DC6H5 -> UFDFPN5_1P7X1P4_STM
- moved R1 10.8 mm to (211.0, 106.7)
- moved R2 10.7 mm to (215.9, 105.4)
- moved R109 9.06 mm to (194.3, 101.6)
- moved D109 9.06 mm to (190.5, 101.6)
- moved R108 7.92 mm to (194.3, 105.4)
- moved D108 7.92 mm to (190.5, 105.4)
- moved R107 6.65 mm to (194.3, 109.2)
- moved D107 6.65 mm to (190.5, 109.2)
- moved R106 5.51 mm to (194.3, 113.0)
- moved D106 5.51 mm to (190.5, 113.0)
- moved C2 4.75 mm to (221.9, 126.8), turned to 90 degrees
- moved R105 4.37 mm to (194.3, 116.8)
- moved D105 4.37 mm to (190.5, 116.8)
- moved R104 3.11 mm to (194.3, 120.7)
- moved D104 3.10 mm to (190.5, 120.7)
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Connections:
- U102 pad 3: Net-(U102-Pad3) -> Net-(L101-Pad1)
- U102 pad 4: Net-(U102-Pad3) -> Net-(L101-Pad2)
Routing:
- net /MOSI: track 0.00 -> 64.1 mm, vias 0 -> 5
- net +3V3: track 0.00 -> 60.6 mm, vias 0 -> 2
- net /MISO: track 0.00 -> 49.6 mm, vias 0 -> 5
- net /SCK: track 0.00 -> 48.0 mm, vias 0 -> 4
- net /LED_0: track 0.00 -> 42.5 mm, vias 0 -> 2
- net /SDA: track 0.00 -> 39.6 mm, vias 0 -> 2
- net /RESET: track 0.00 -> 39.5 mm, vias 0 -> 2
- net /SCL: track 0.00 -> 38.6 mm, vias 0 -> 2
- net GND: track 0.00 -> 34.9 mm, vias 0 -> 21
- net /TOUCH_RECEIVE: track 0.00 -> 34.0 mm, vias 0 -> 2
- net /LED_1: track 0.00 -> 33.6 mm
- net /LED_2: track 0.00 -> 30.1 mm
- net /LED_3: track 0.00 -> 27.5 mm
- net /LED_4: track 0.00 -> 25.0 mm
- net /LED_5: track 0.00 -> 23.1 mm
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Other:
- outline, holes or cut-outs redrawn
- board text added: "1. Insert battery where the positive side contacts the + and negative contacts the -"
- board text added: "2. Hold the card such that the LED strip is parallel to your arm and your fingers are near the battery."
- board text added: "3. Shake the card 2-3 times per second from left to right"
- board text added: "Instructions:"

Commit message: Preparing version 4 for manufacture
Parts:
- ICSP1: moved to B.Cu
- moved ICSP1 2.63 mm to (230.4, 84.3), turned to 90 degrees
- moved C2 1.94 mm to (220.0, 126.8)
- moved R3 1.94 mm to (220.0, 130.0)
Routing:
- net /MOSI: track 64.1 -> 67.8 mm, vias 5 -> 6
- net /RESET: track 39.5 -> 36.8 mm
- net /MISO: track 49.6 -> 47.0 mm, vias 5 -> 4
- net /SCK: track 48.0 -> 46.4 mm
- net /TOUCH_RECEIVE: track 34.0 -> 34.9 mm
Other:
- board text removed: "1. Insert battery where the positive side contacts the + and negative contacts the -"
- board text removed: "2. Hold the card such that the LED strip is parallel to your arm and your fingers are near the battery."
- board text removed: "3. Shake the card 2-3 times per second from left to right"
- board text removed: "Instructions:"
