File: design/business_card/business_card.kicad_sch (KiCad schematic)
At the start: 33 parts, among them U101 ATtiny861A-M, U102 ST25TA02KB-DC6H5, U103 LIS3DHTR

Commit message: Routing complete
Parts:
- added L101: 2.75uH, CustomFootprints:Trace_Inductor_2_75uH, symbol pspice:INDUCTOR
Connections:
- net at U102.3 (AC0): now also L101.1; no longer U102.4 (AC1)
- new net: L101.2, U102.4 (AC1)
Changed lines of the file:
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@@
     (stroke (width 0) (type solid) (color 0 0 0 0))
   )
-  (wire (pts (xy 204.47 101.6) (xy 210.185 101.6))
+  (wire (pts (xy 204.47 101.6) (xy 206.375 101.6))
+    (stroke (width 0) (type solid) (color 0 0 0 0))
+  )
+  (wire (pts (xy 204.47 104.14) (xy 206.375 104.14))
+    (stroke (width 0) (type solid) (color 0 0 0 0))
+  )
+  (wire (pts (xy 206.375 95.885) (xy 212.09 95.885))
+    (stroke (width 0) (type solid) (color 0 0 0 0))
+  )
+  (wire (pts (xy 206.375 101.6) (xy 206.375 95.885))
+    (stroke (width 0) (type solid) (color 0 0 0 0))
+  )
+  (wire (pts (xy 206.375 104.14) (xy 206.375 108.585))
+    (stroke (width 0) (type solid) (color 0 0 0 0))
+  )
+  (wire (pts (xy 206.375 108.585) (xy 212.09 108.585))
     (stroke (width 0) (type solid) (color 0 0 0 0))
   )
@@
   )
   (wire (pts (xy 208.28 70.485) (xy 208.28 73.025))
-    (stroke (width 0) (type solid) (color 0 0 0 0))
-  )
-  (wire (pts (xy 210.185 88.9) (xy 214.63 88.9))
-    (stroke (width 0) (type solid) (color 0 0 0 0))
-  )
-  (wire (pts (xy 210.185 101.6) (xy 210.185 88.9))
-    (stroke (width 0) (type solid) (color 0 0 0 0))
-  )
-  (wire (pts (xy 210.185 104.14) (xy 204.47 104.14))
-    (stroke (width 0) (type solid) (color 0 0 0 0))
-  )
-  (wire (pts (xy 210.185 116.84) (xy 210.185 104.14))
-    (stroke (width 0) (type solid) (color 0 0 0 0))
-  )
-  (wire (pts (xy 214.63 88.9) (xy 214.63 116.84))
-    (stroke (width 0) (type solid) (color 0 0 0 0))
-  )
-  (wire (pts (xy 214.63 116.84) (xy 210.185 116.84))
     (stroke (width 0) (type solid) (color 0 0 0 0))
   )
@@
     )
     (property "Datasheet" "~" (id 3) (at 270.51 56.515 0)
+      (effects (font (size 1.27 1.27)) hide)
+    )
+    (pin "1")
+    (pin "2")
+  )
+  (symbol (lib_id "pspice:INDUCTOR") (at 212.09 102.235 90) (unit 1)
+    (in_bom yes) (on_board yes)
+    (property "Reference" "L101" (id 0) (at 213.995 100.965 90)
+      (effects (font (size 1.27 1.27)) (justify right))
+    )
+    (property "Value" "2.75uH" (id 1) (at 207.01 93.345 90)
+      (effects (font (size 1.27 1.27)) (justify right))
+    )
+    (property "Footprint" "CustomFootprints:Trace_Inductor_2_75uH" (id 2) (at 212.09 102.235 0)
+      (effects (font (size 1.27 1.27)) hide)
+    )
+    (property "Datasheet" "~" (id 3) (at 212.09 102.235 0)
       (effects (font (size 1.27 1.27)) hide)
     )
@@
       (reference "ICSP1") (unit 1) (value "ICSP") (footprint "Connector_PinHeader_2.54mm:PinHeader_2x03_P2.54mm_Vertical")
     )
+    (path "/4189afe8-8da3-4794-929d-bf750375b842"
+      (reference "L101") (unit 1) (value "2.75uH") (footprint "CustomFootprints:Trace_Inductor_2_75uH")
+    )
     (path "/00000000-0000-0000-0000-00005c0ecd2e"

Commit message: Deleted kicad session file, tested image_to_laser
Parts:
- C1, C101: Digikey (none) -> 1276-6456-1-ND
- C102: Digikey (none) -> 311-1779-1-ND
- C2: Digikey (none) -> 732-7762-1-ND
- D101, D102, D103, D104, D105, D106, D107, D108, D109: Digikey (none) -> 160-1183-1-ND
- R1, R2: Digikey (none) -> 311-10KGRCT-ND
- R101, R102, R103, R104, R105, R106, R107, R108, R109: Digikey (none) -> 311-240GRCT-ND
- R3: Digikey (none) -> 311-976KHRCT-ND
- U101: Digikey (none) -> ATTINY861-15MZCT-ND
- U102: Digikey (none) -> 497-19639-1-ND
